File: hardware/mainboard/mainboard.kicad_pcb (KiCad board)
At the start: 4 copper layers, 180 x 75 mm, 330 parts, among them J1 USB 2.0, J10 JST XH, J11 JST XH, J12 EXP1, J13 EXP2, J14 JST XH, J15 JST XH, J16 JST XH, J17 JST XH, J18 JST XH, J19 JST XH, J2 JST XH, J20 Screw_Terminal_01x02, J21 Screw_Terminal_01x02, J22 Screw_Terminal_01x02, J23 Screw_Terminal_01x02, J24 Conn_01x05_Pin, J25 FPC 8p 0.5mm, J26 USB_A_Stacked, J27 USB_A_Stacked, J3 Power In, J4 JST XH, J5 JST XH, J6 JST XH, J7 JST XH, J8 JST XH, J9 JST XH, M1 JST XH, M2 JST XH, M3 JST XH, M4 JST XH, M5 Micro-Fit 3.0, M6 Micro-Fit 3.0, Q1 AGM308MBP, Q10 DMT6016, Q11 DMT6016, Q12 DMT6016, Q13 DMT6016, Q14 DMT6016, Q15 DMT6016, Q16 DMT6016, Q17 DMT6016, Q18 DMT6016, Q19 DMT6016, Q2 AGM308MBP, Q20 AGM308MBP, Q21 AGM308MBP, Q22 AGM308MBP, Q23 AGM308MBP, Q24 AGM308MBP, Q25 AGM308MBP, Q26 AGM308MBP, Q3 AGM308MBP, Q4 DMT6016, Q5 DMT6016, Q6 DMT6016, Q7 DMT6016, Q8 DMT6016, Q9 DMT6016, SW1 SW_SPDT, SW2 SW_SPDT, SW3 SPDT, 2A, SW4 SPDT, 2A, SW5 SPDT, 2A, SW6 SPDT, 2A, SW7 SPDT, 2A, SW8 SPDT, 2A, SW9 SW_SPDT, T1 V_{SA}, T10 TestPoint, T11 TestPoint, T12 TestPoint, T13 TestPoint, T14 TestPoint, T15 TestPoint, T16 TestPoint, T17 V_{SA}, T18 SClk, T19 Gnd, T2 SClk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

Commit message: added components and further work on PCB layout design
Parts:
- added H5: V_{M}, corevus:M3_M2.5_PCB_Nut, F.Cu at (90.0, 36.0)
- C38, C40, C53, C55: value 47nF 100V/2 -> 47nF 50V
- C44, C46, C59, C61: value 100nF 63V/2 -> 100nF 50V
- C51, C52, C66, C67: value 1μF 63V -> 1μF 100V
- Q10, Q11, Q12, Q13, Q14, Q15, Q16, Q17, Q18, Q19, Q4, Q5, Q6, Q7, Q8, Q9: value DMT6016 -> DMT6016LFDF
- U11, U12: footprint Package_QFP:TQFP-48-1EP_7x7mm_P0.5mm_EP5x5mm_ThermalVias -> corevus:TMCx160
- moved J24 178.8 mm to (143.9, 82.0), turned to 90 degrees
- moved J19 55.7 mm to (92.0, 105.0)
- moved C33 36.8 mm to (167.6, 53.5), turned to -90 degrees
- moved C34 35.3 mm to (160.0, 54.2)
- moved C35 32.3 mm to (160.0, 53.2), turned to 180 degrees
- moved C36 29.3 mm to (160.0, 52.2), turned to 180 degrees
- moved R28 26.2 mm to (160.0, 51.2)
- moved C37 23.2 mm to (170.5, 49.0), turned to 90 degrees
- moved T5 22.5 mm to (105.2, 63.5), turned to 180 degrees
- moved T6 22.2 mm to (109.8, 63.5), turned to 180 degrees
- moved T1 22.1 mm to (102.2, 63.5), turned to 180 degrees
- moved T3 22.1 mm to (106.8, 63.5), turned to 180 degrees
- moved T2 22.1 mm to (103.8, 63.5), turned to 180 degrees
- moved T4 22.1 mm to (108.2, 63.5), turned to 180 degrees
- moved Q26 21.4 mm to (84.7, 105.6)
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Connections:
- F1 pad 1: VMC -> Net-(J3-Pin_2)
- F1 pad 2: Net-(J3-Pin_2) -> VMC
- F2 pad 1: VMC -> Net-(J3-Pin_4)
- F2 pad 2: Net-(J3-Pin_4) -> VMC
- F3 pad 1: /Bed_H+ -> Net-(J3-Pin_4)
- F3 pad 2: Net-(J3-Pin_4) -> /Bed_H+
- F4 pad 1: VMB -> Net-(J3-Pin_2)
- F4 pad 2: Net-(J3-Pin_2) -> VMB
- F5 pad 1: VMB -> Net-(J3-Pin_4)
- F5 pad 2: Net-(J3-Pin_4) -> VMB
- F6 pad 1: +24V -> Net-(J3-Pin_4)
- F6 pad 2: Net-(J3-Pin_4) -> +24V
Routing:
- net /_{M20}Step: track 0.00 -> 75.9 mm
- net +12V: track 8.63 -> 80.9 mm, vias 0 -> 2
- net /SClk_{3}: track 0.00 -> 70.8 mm, vias 0 -> 3
- net +3.3V: track 0.00 -> 70.7 mm, vias 0 -> 2
- net /_{M22}Step: track 0.00 -> 70.0 mm
- net /_{M22}~{CS}: track 0.00 -> 69.9 mm
- net /MOSI_{3}: track 0.00 -> 69.8 mm, vias 0 -> 4
- net /_{M22}Dir: track 0.00 -> 67.2 mm
- net /_{M22}~{En}: track 0.00 -> 66.7 mm
- net /MISO_{3}: track 0.00 -> 65.8 mm, vias 0 -> 3
- net /_{M12}Step: track 0.00 -> 57.7 mm
- net /_{M12}Dir: track 0.00 -> 54.9 mm
- net /_{M12}~{En}: track 0.00 -> 53.7 mm
- net /_{M20}Dir: track 0.00 -> 53.5 mm
- net /_{M12}~{CS}: track 0.00 -> 53.1 mm
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- added copper zone on F.Cu, net +24V
- added copper zone on B.Cu, net /Bed_H+
- added copper zone on F.Cu, net /Bed_H+
- added copper zone on F.Cu, net /Motor 3 (TMC2208)/A1
- added copper zone on F.Cu, net /Motor 3 (TMC2208)/A2
- added copper zone on F.Cu, net /Motor 3 (TMC2208)/B1
- added copper zone on F.Cu, net /Motor 3 (TMC2208)/B2
- added copper zone on F.Cu, net /Motor 3 (TMC2208)/BRA
- added copper zone on F.Cu, net /Motor 3 (TMC2208)/BRB
- added copper zone on B.Cu, net Net-(J3-Pin_2)
- added copper zone on F.Cu, net Net-(J3-Pin_2)
- added copper zone on B.Cu, net Net-(J3-Pin_4)
- added copper zone on F.Cu, net Net-(J3-Pin_4)
- added copper zone on B.Cu, net Net-(Q11-S-Pad4)
- added copper zone on In2.Cu, net Net-(Q11-S-Pad4)
- added copper zone on B.Cu, net Net-(Q13-S-Pad4)
- added copper zone on In2.Cu, net Net-(Q13-S-Pad4)
- added copper zone on B.Cu, net Net-(Q17-S-Pad4)
- added copper zone on F.Cu, net Net-(Q17-S-Pad4)
- added copper zone on In2.Cu, net Net-(Q17-S-Pad4)
- added copper zone on B.Cu, net Net-(Q5-S-Pad4)
- added copper zone on In2.Cu, net Net-(Q5-S-Pad4)
- added copper zone on B.Cu, net VMB
- added copper zone on In2.Cu, net VMB
- added copper zone on B.Cu, net VMC
- added copper zone on In2.Cu, net VMC
Other:
- outline, holes or cut-outs redrawn
- board text added: "1"
