File: hardware/mainboard/mainboard.kicad_sch (KiCad schematic)
At the start: 54 parts, among them J1 USB 2.0, J10 JST XH, J11 JST XH, J12 JST XH, J2 USB_A, J3 JST XH, J4 JST XH, J5 JST XH, J6 JST XH, J7 JST XH, J8 JST XH, J9 Power Delivery, Q1 NMOS, SW1 DFU, SW2 Reset, SW3 SPDT, 2A, U1 STM32F446ZCTx, U8 4504, Y1 12 MHz

Commit message: added fan / heater ports to mainboard, and footprints for switches, transistors, etc.
Parts:
- removed H1: VM, corevus:M4_PCB_Nut, symbol Mechanical:MountingHole_Pad
- removed H2, H4, H6: Gnd, corevus:M4_PCB_Nut, symbol Mechanical:MountingHole_Pad
- removed H3: Supply, corevus:M4_PCB_Nut, symbol Mechanical:MountingHole_Pad
- removed H5: Bed Supply, corevus:M4_PCB_Nut, symbol Mechanical:MountingHole_Pad
- removed H7: Bed Out, corevus:M4_PCB_Nut, symbol Mechanical:MountingHole_Pad
- removed H8: Bed Return, corevus:M4_PCB_Nut, symbol Mechanical:MountingHole_Pad
- removed J12: JST XH, symbol Connector:Conn_01x02_Pin
- removed J2: USB_A, symbol Connector:USB_A
- removed J7, J8: JST XH, symbol Connector:Conn_01x03_Pin
- removed Q1: NMOS, symbol Device:Q_NMOS_DGS
- removed R3 (x2): 27Ω, symbol Device:R_Small
- removed SW1: DFU, symbol Switch:SW_SPST
- removed SW3: SPDT, 2A, symbol Switch:SW_SPDT
- added D1 (x2): A, AlphaLib:0603LED, symbol Device:LED_Small
- added FID1, FID2, FID3, FID4, FID5, FID6: Fiducial, Fiducial:Fiducial_0.5mm_Mask1mm, symbol Mechanical:Fiducial
- added H1, H2, H3, H4: MountingHole, MountingHole:MountingHole_3.2mm_M3_Pad_Via, symbol Mechanical:MountingHole
- added Q1 (x2): AGM308MBP, corevus:AGM308MBP, symbol Device:Q_Dual_NMOS_S1G1S2G2D2D2D1D1
- added R3 (x2): 1kΩ, AlphaLib:0603R, symbol Device:R_Small
- added R3: 10kΩ, AlphaLib:0603R, symbol Device:R_Small
- added SW14: SW_SPDT, symbol Switch:SW_SPDT
- added SW9: SW_SPDT, corevus:MSS12C02-LS, symbol Switch:SW_SPDT
- added U9: 4504, Package_SO:SOIC-16_3.9x9.9mm_P1.27mm, symbol 4xxx:4504
- J10, J11, J3, J4, J5, J6: footprint (none) -> Connector_JST:JST_XH_B3B-XH-A_1x03_P2.50mm_Vertical
- J9: footprint (none) -> corevus:DBT50G-9.5-6P
- U8: footprint (none) -> Package_SO:SOIC-16_3.9x9.9mm_P1.27mm
Connections:
- net Heatbed is gone; now on net +24V: J9.6 (Pin_6)
- net +12V: now also U8.16 (VDD), U9.16 (VDD)
- net +3.3V: now also SW14.3 (C)
- net BOOT0: now also SW14.2 (B)
- net GND: now also Q1.1 (S), Q1.1 (S), Q1.3 (S), Q1.3 (S), R3.2, R3.2, R3.2, SW14.1 (A), SW9.1 (A), U9.8 (VSS); no longer J9.5 (Pin_5)
- net Fan3_Gate: now reaches U8.10 (Dout)
- net Fan4_Gate: now reaches U8.12 (Eout)
- net Fan5_Gate: now reaches U8.15 (Fout)
- net Fan0_Gate: now reaches U8.2 (Aout)
- net Fan1_Gate: now reaches U8.4 (Bout)
- net Fan2_Gate: now reaches U8.6 (Cout)
- new net: D1.1 (K), R3.1 (x2)
- new net: D1.2 (A), Q1.2 (G), Q1.2 (G), Q1.4 (G), Q1.4 (G), R3.1, SW9.2 (B)
- new net Bed_Gate: D1.2 (A), SW9.3 (C), U9.15 (Fout)
- new net Bed_H-: J9.5 (Pin_5), Q1.5 (D), Q1.5 (D), Q1.6 (D), Q1.6 (D), Q1.7 (D), Q1.7 (D), Q1.8 (D), Q1.8 (D)
- new net HE0_Gate: U9.2 (Aout)
- new net HE1_Gate: U9.4 (Bout)
- new net HE2_Gate: U9.6 (Cout)
Other:
- added sheet Fans 0, 1 (driver-fan-2pin-dual.kicad_sch)
- added sheet Fans 2, 3 (driver-fan-2pin-dual.kicad_sch)
- added sheet Fans 4, 5 (driver-fan-2pin-dual.kicad_sch)
- added sheet Heater 0 (driver_heater.kicad_sch)
- added sheet Heater 1 (driver_heater.kicad_sch)
- added sheet Heater 2 (driver_heater.kicad_sch)
- added sheet Raspberry Pi Zero (pi-zero.kicad_sch)
- note added: "2x2 7mΩ FETs dissipate ~110 mW at 8A."
- note added: "Mechanical switch hard-cutoffs gate drive signal and shorts it to ground."
- note removed: "ADD JUMPER TO ENABLE ALL POWER MOSFETS FOR BED / HOTEND HEATERS"
- note removed: "HIGH SIDE BED MOSFET"
- note removed: "Power Delivery"
- moved on the sheet: C10, SW2, U8

Commit message: saving mainboard, gonna tear out the entire thing and redo in 4-layer
Parts:
- removed Q1: AGM308MBP, corevus:AGM308MBP, symbol Device:Q_Dual_NMOS_S1G1S2G2D2D2D1D1
- removed R3 (x2): 27Ω, symbol Device:R_Small
- added D1: A, AlphaLib:0603LED, symbol Device:LED_Small
- added F6: 10A, corevus:XF-508P-B, symbol Device:Fuse
- added Q1 (x2): AGM308MBP, corevus:AGM308MBP, symbol Device:Q_Dual_NMOS_S1G1S2G2D2D2D1D1
- added R3: 1kΩ, AlphaLib:0603R, symbol Device:R_Small
- added R3 (x2): 33Ω, AlphaLib:0402R, symbol Device:R_Small
- C27, C33, C7, C9: footprint Capacitor_SMD:CP_Elec_16x17.5 -> Capacitor_THT:CP_Radial_D12.5mm_P5.00mm
- F1, F2, F3, F4, F5: footprint Fuse:Fuse_Blade_ATO_directSolder -> corevus:XF-508P-B
- J1: footprint (none) -> Connector_USB:USB_C_Receptacle_XKB_U262-16XN-4BVC11
- J9: value Power Delivery -> Power In
- SW14: footprint (none) -> corevus:MSS12C02-LS
Connections:
- net +5V is gone; now on net +3.3V: J10.1 (Pin_1), J11.1 (Pin_1), J3.1 (Pin_1), J4.1 (Pin_1), J5.1 (Pin_1), J6.1 (Pin_1)
- net VMA is gone; now on net +24V: C6.1, C8.1, F1.2
- net +24V: no longer F1.1, J9.4 (Pin_4), J9.6 (Pin_6)
- net +48V: now also F3.1, F5.1, J9.1 (Pin_1); no longer F3.2, F5.2, J9.2 (Pin_2)
- net BOOT0: now also D1.2 (A)
- net Bed_Gate: now also SW9.1 (A); no longer SW9.3 (C)
- net Bed_H-: now also J9.6 (Pin_6), Q1.5 (D), Q1.5 (D), Q1.6 (D), Q1.6 (D), Q1.7 (D), Q1.7 (D), Q1.8 (D), Q1.8 (D); no longer J9.5 (Pin_5)
- net GND: now also J9.2 (Pin_2), J9.4 (Pin_4), SW9.3 (C), U1.107 (VSS), U1.120 (VSS), U1.130 (VSS), U1.16 (VSS), U1.38 (VSS), U1.51 (VSS), U1.61 (VSS), U1.83 (VSS), U1.94 (VSS), Q1.1 (S), Q1.1 (S), Q1.3 (S), Q1.3 (S), R3.1; no longer J9.1 (Pin_1), J9.3 (Pin_3), SW9.1 (A)
- net USB_D+: now also R3.1
- net USB_D-: now also R3.1
- net VMB: now also C33.1, F3.2; no longer C7.1, F3.1
- net VMC: now also C7.1, F5.2; no longer C33.1, F5.1
- net BG: now reaches D1.2 (A), Q1.2 (G), Q1.4 (G), R3.1, SW9.2 (B)
- net BG: now also Q1.2 (G), Q1.2 (G), Q1.4 (G), Q1.4 (G)
- net at J1.A6 (D+), J1.B6 (D+): now also R3.2
- net at J1.A7 (D-), J1.B7 (D-): now also R3.2
- net HE3_Gate: now reaches U9.10 (Dout)
- new net: F1.1, F6.2, J9.3 (Pin_3)
- new net: D1.1 (K), R3.2
- new net Bed_H+: F6.1, J9.5 (Pin_5)
Other:
- added sheet Heater 3 (driver_heater.kicad_sch)
- added sheet Motor Expansion 2x (driver_expansion.kicad_sch)
- sheet Motor Expansion 1x ports: added Clk, MISO, MOSI, SClk, V_{CC}IO, V_{M}, V_{SA}, _{M0}Diag0, _{M0}Diag1, _{M0}Dir, _{M0}Step, _{M0}~{CS}, _{M0}~{En}, _{M2}Diag0, _{M2}Diag1, _{M2}Dir, _{M2}Step, _{M2}~{CS}, _{M2}~{En}; removed none
- note added: "3x2 7mΩ FETs dissipate ~50 mW at 8A."
- note removed: "2x2 7mΩ FETs dissipate ~110 mW at 8A."
- moved on the sheet: C10, F3, F5, FID1, FID2, FID3, FID4, FID5, FID6, Q1B, R3, SW14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

Commit message: further board edits, mostly done with power planes, heaters, fans, motor channels, starting work on microcontroller signals
Parts:
- removed D1 (x2): A, AlphaLib:0603LED, symbol Device:LED_Small
- removed J10, J11: JST XH, Connector_JST:JST_XH_B3B-XH-A_1x03_P2.50mm_Vertical, symbol Connector:Conn_01x03_Pin
- removed R3 (x2): 1kΩ, AlphaLib:0603R, symbol Device:R_Small
- removed R3: 10kΩ, AlphaLib:0603R, symbol Device:R_Small
- removed U1: STM32F446ZCTx, Package_QFP:LQFP-144_20x20mm_P0.5mm, symbol MCU_ST_STM32F4:STM32F446ZCTx
- added C10: 22μF, Capacitor_SMD:C_1206_3216Metric, symbol Device:C_Small
- added C10: 330pF, AlphaLib:0402C, symbol Device:C_Small
- added C10: 100nF, AlphaLib:0402C, symbol Device:C_Small
- added C10: 1nF, AlphaLib:0402C, symbol Device:C_Small
- added C10 (x5): 1μF, AlphaLib:0402C, symbol Device:C_Small
- added C10: μF, AlphaLib:0402C, symbol Device:C_Small
- added C10: 10μF, Capacitor_SMD:C_1206_3216Metric, symbol Device:C_Small
- added C10: 26nF, AlphaLib:0402C, symbol Device:C_Small
- added C72, C78: 330μF 35V, Capacitor_SMD:CP_Elec_8x10, symbol Device:C_Polarized_Small_US
- added D1 (x2): A, AlphaLib:0603LED, symbol Device:LED_Small
- added D1: G, symbol Device:LED_Small
- added J10: EXP1, Connector_IDC:IDC-Header_2x05_P2.54mm_Vertical, symbol Connector_Generic:Conn_02x05_Odd_Even
- added J11: EXP2, Connector_IDC:IDC-Header_2x05_P2.54mm_Vertical, symbol Connector_Generic:Conn_02x05_Odd_Even
- added J22: SPI-something, Connector_IDC:IDC-Header_2x05_P2.54mm_Vertical, symbol Connector_Generic:Conn_02x05_Odd_Even
- added J23, J25, J26, J27: JST XH, Connector_JST:JST_XH_B2B-XH-A_1x02_P2.50mm_Vertical, symbol Connector:Conn_01x02_Pin
- added J24: JST XH, Connector_JST:JST_XH_B3B-XH-A_1x03_P2.50mm_Vertical, symbol Connector:Conn_01x03_Pin
- added L1: 4.7μH, Inductor_SMD:L_Sunlord_MWSA1004S, symbol Device:L
- added Q1: AGM308MBP, corevus:AGM308MBP, symbol Device:Q_Dual_NMOS_S1G1S2G2D2D2D1D1
- added R3 (x4): 4.7kΩ, AlphaLib:0402R, symbol Device:R_Small
- added R3: 2.41kΩ, AlphaLib:0402R, symbol Device:R_Small
- added R3 (x3): 1kΩ, AlphaLib:0402R, symbol Device:R_Small
- added R3 (x3): Ω, symbol Device:R_Small
- added R3: 100kΩ, AlphaLib:0402R, symbol Device:R_Small
- added R3 (x2): 200kΩ, symbol Device:R_Small
- added R3 (x2): Ω, AlphaLib:0402R, symbol Device:R_Small
- added R3: 10kΩ, AlphaLib:0402R, symbol Device:R_Small
- added SW13: SW_SPDT, corevus:MSS12C02-LS, symbol Switch:SW_SPDT
- added U1: STM32F407VGTx, Package_QFP:LQFP-100_14x14mm_P0.5mm, symbol MCU_ST_STM32F4:STM32F407VGTx
- added U11: NCP3011, Package_SO:TSSOP-14_4.4x5mm_P0.65mm, symbol corevus:NCP3011
- C10: value xyzpF -> 20pF
Connections:
- net +12V: now also C10.1, C10.2, C78.1, D1.2 (A), L1.2, R3.1
- net +24V: now also C10.2, C72.1, Q1.5 (D), Q1.6 (D), R3.1, U11.14 (V_{CC}); no longer F2.1, F4.1
- net +3.3V: now also R3.2, R3.2, R3.2, R3.2
- net +48V: now also J9.2 (Pin_2), R3.1; no longer J9.1 (Pin_1)
- net BG: now also D1.2 (A), R3.1
- net BOOT0: now also U1.94 (BOOT0)
- net Bed_Gate: now also D1.2 (A)
- net GND: now also J9.1 (Pin_1), J9.3 (Pin_3), C10.1, C10.1, C10.1, C10.1, C10.1, C10.1, C10.1, C10.1, C10.1, C72.2, C78.2, J23.2 (Pin_2), J25.2 (Pin_2), J26.2 (Pin_2), J27.2 (Pin_2), Q1.1 (S), R3.1, R3.1, R3.1, R3.2, R3.2, R3.2, R3.2, R3.2, R3.2, R3.2, U1.10 (VSS), U1.20 (VSSA), U1.27 (VSS), U1.74 (VSS), U1.99 (VSS), U11.8 (Gnd); no longer J9.2 (Pin_2), J9.4 (Pin_4)
- net MISO_{1}: now also U1.31 (PA6)
- net MOSI_{1}: now also U1.32 (PA7)
- net SClk_{1}: now also U1.30 (PA5)
- net USB_D+: now also U1.71 (PA12)
- net USB_D-: now also U1.70 (PA11)
- net ~{Reset}: now also U1.14 (NRST)
- net at C10.2, R3.2, Y1.3: now also U1.13 (PH1)
- net at F1.1, F6.2: now also F2.1, F4.1, J9.4 (Pin_4); no longer J9.3 (Pin_3)
- net at C10.2, R3.1, Y1.1: now also U1.12 (PH0)
- new net: C10.1, R3.2
- new net: C10.1, L1.1, Q1.3 (S), Q1.7 (D), Q1.8 (D), R3.2, U11.11 (VSw)
- new net: Q1.4 (G), R3.1, U11.12 (HSDr)
- new net: D1.1 (K), R3.1 (x2)
- new net: C10.2, C10.2, U11.6 (Comp)
- new net: R3.1, R3.2, R3.2, U11.7 (FB)
- new net: C10.2, R3.2, U11.1 (VRef)
- new net: C10.2, U11.2 (En)
- new net: C10.2, R3.1
- new net: Q1.2 (G), R3.1, U11.9 (LSDr)
- new net: C10.2, U11.13 (BSt)
- new net: D1.1 (K), R3.2
- new net Th_{0}: C10.2, J23.1 (Pin_1), R3.1, U1.15 (PC0)
- new net Th_{1}: C10.2, J25.1 (Pin_1), R3.1, U1.16 (PC1)
- new net Th_{2}: C10.2, J26.1 (Pin_1), R3.1, U1.17 (PC2)
- new net Th_{3}: C10.2, J27.1 (Pin_1), R3.1, U1.18 (PC3)
- new net USART_{1}_RX: U1.69 (PA10)
- new net USART_{1}_TX: U1.68 (PA9)
- no-connect marks 6 -> 8
Other:
- sheet Raspberry Pi Zero renamed Pi Zero + USB Hub
- note added: "24→12V Step-Down"
- note added: "Capacitor dissipation resistors"
- note added: "I spend good f*cking money on this IC so y'all better use it"
- note removed: "Endstop ports may be used to drive 5-volt Neopixel-style LED chains or fans. Due to lack of LED pinout standardization, you may need to (re)crimp connectors."
- moved on the sheet: C10, D1, F1, F2, F3, F4, F5, F6, J1, R3, SW14, SW2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

Commit message: redid mainboard, added probe wiring, replacing ncp chip with LM5160 for now
Parts:
- removed C10: 22μF, Capacitor_SMD:C_1206_3216Metric, symbol Device:C_Small
- removed C10: 330pF, AlphaLib:0402C, symbol Device:C_Small
- removed C10: 100nF, AlphaLib:0402C, symbol Device:C_Small
- removed C10: 10μF, symbol Device:C_Small
- removed C10: 1nF, AlphaLib:0402C, symbol Device:C_Small
- removed C10: 1μF, AlphaLib:0402C, symbol Device:C_Small
- removed C10: μF, AlphaLib:0402C, symbol Device:C_Small
- removed C10: 10μF, Capacitor_SMD:C_1206_3216Metric, symbol Device:C_Small
- removed C10: 26nF, AlphaLib:0402C, symbol Device:C_Small
- removed C72, C78: 330μF 35V, Capacitor_SMD:CP_Elec_8x10, symbol Device:C_Polarized_Small_US
- removed D1: A, symbol Device:LED_Small
- removed D1: G, symbol Device:LED_Small
- removed Q1: AGM308MBP, corevus:AGM308MBP, symbol Device:Q_Dual_NMOS_S1G1S2G2D2D2D1D1
- removed R3: 2.41kΩ, AlphaLib:0402R, symbol Device:R_Small
- removed R3: 1kΩ, symbol Device:R_Small
- removed R3 (x3): Ω, symbol Device:R_Small
- removed R3: 100kΩ, AlphaLib:0402R, symbol Device:R_Small
- removed R3 (x2): Ω, AlphaLib:0402R, symbol Device:R_Small
- removed R3: 1kΩ, AlphaLib:0402R, symbol Device:R_Small
- removed U11: NCP3011, Package_SO:TSSOP-14_4.4x5mm_P0.65mm, symbol corevus:NCP3011
- removed U8, U9: 4504, Package_SO:SOIC-16_3.9x9.9mm_P1.27mm, symbol 4xxx:4504
- added C10 (x4): 1μF, AlphaLib:0603C, symbol Device:C_Small
- added C10 (x2): 10nF, AlphaLib:0402C, symbol Device:C_Small
- added C10 (x2): 1μF, AlphaLib:0402C, symbol Device:C_Small
- added C10: 100nF, AlphaLib:0402C, symbol Device:C_Small
- added C10 (x2): 1nF, AlphaLib:0402C, symbol Device:C_Small
- added C10 (x2): 50nF, AlphaLib:0402C, symbol Device:C_Small
- added C10 (x2): 22μF, Capacitor_SMD:C_0805_2012Metric, symbol Device:C_Small
- added C10 (x2): 3.3nF, AlphaLib:0402C, symbol Device:C_Small
- added D1 (x2): G, AlphaLib:0603LED, symbol Device:LED_Small
- added L2: 15μH/3A, Inductor_SMD:L_Chilisin_BMRB00060618, symbol Device:L
- added R3 (x2): 10kΩ, AlphaLib:0402R, symbol Device:R_Small
- added R3 (x4): 150kΩ, AlphaLib:0402R, symbol Device:R_Small
- added R3: 3.3kΩ, AlphaLib:0402R, symbol Device:R_Small
- added R3 (x2): 100kΩ, AlphaLib:0402R, symbol Device:R_Small
- added R3 (x4): 1kΩ, AlphaLib:0402R, symbol Device:R_Small
- added R3: 5.1kΩ, AlphaLib:0402R, symbol Device:R_Small
- added R3: 2.2kΩ, AlphaLib:0402R, symbol Device:R_Small
- added R3: 200Ω, AlphaLib:0402R, symbol Device:R_Small
- added R3: 220kΩ, AlphaLib:0402R, symbol Device:R_Small
- added U11, U8: LM5160A, Package_SON:WSON-12-1EP_4x4mm_P0.5mm_EP2.6x3mm_ThermalVias, symbol corevus:LM5160A
- added U12, U13, U9: CD40109B, Package_SO:TSSOP-16_4.4x5mm_P0.65mm, symbol corevus:CD40109B
- added U14: LTV-357T, Package_SO:SO-4_4.4x3.6mm_P2.54mm, symbol Isolator:LTV-357T
- C10: footprint (none) -> AlphaLib:0402C
- L1: value 4.7μH -> 15μH/3A; footprint Inductor_SMD:L_Sunlord_MWSA1004S -> Inductor_SMD:L_Chilisin_BMRB00060618; LCSC (none) -> C475522
- R3: footprint (none) -> AlphaLib:0402R
- R3: footprint AlphaLib:0603R -> AlphaLib:0402R
- R3: value xyzkΩ -> kΩ; footprint (none) -> AlphaLib:0402R
- SW2: footprint (none) -> Button_Switch_SMD:SW_SPST_SKQG_WithStem
- Y1: footprint (none) -> Crystal:Crystal_SMD_3225-4Pin_3.2x2.5mm
Connections:
- net +12V: now also C10.1, C10.1, D1.2 (A), R3.1, U12.16 (V_{DD}), U13.16 (V_{DD}), U9.16 (V_{DD})
- net +24V: now also SW13.3 (C), C10.1, C10.1, C10.1, C10.1, R3.1, R3.1, R3.2, R3.2, U11.3 (VIn), U8.3 (VIn)
- net +3.3V: now also U1.100 (VDD), U1.11 (VDD), U1.19 (VDD), U1.22 (VDDA), U1.28 (VDD), U1.50 (VDD), U1.6 (VBAT), U1.75 (VDD), R3.2, U12.1 (V_{CC}), U12.15 (En_{D}), U12.2 (En_{A}), U12.7 (En_{B}), U12.9 (En_{C}), U13.1 (V_{CC}), U13.15 (En_{D}), U13.2 (En_{A}), U13.7 (En_{B}), U13.9 (En_{C}), U9.1 (V_{CC}), U9.15 (En_{D}), U9.2 (En_{A}), U9.7 (En_{B}), U9.9 (En_{C})
- net Bed_Gate: now also U9.13 (H)
- net Fan0_Gate: now also U9.4 (E)
- net Fan1_Gate: now also U9.5 (F)
- net Fan2_Gate: now also U12.4 (E)
- net Fan3_Gate: now also U12.5 (F)
- net Fan4_Gate: now also U13.4 (E)
- net Fan5_Gate: now also U13.5 (F)
- net GND: now also J24.2 (Pin_2), C10.1, C10.1, C10.1, C10.1, C10.2, C10.2, C10.2, C10.2, C10.2, C10.2, C10.2, R3.1, R3.1, R3.2, R3.2, R3.2, R3.2, R3.2, U11.1 (AGnd), U11.13 (EP), U11.2 (PGnd), U12.8 (V_{SS}), U13.8 (V_{SS}), U14.2, U8.1 (AGnd), U8.13 (EP), U8.2 (PGnd), U9.8 (V_{SS})
- net HE0_Gate: now also U12.13 (H)
- net HE1_Gate: now also U12.11 (G)
- net HE2_Gate: now also U13.13 (H)
- net HE3_Gate: now also U13.11 (G)
- net at L1.1: now also C10.2, R3.1, U11.11 (Sw), U11.12 (Sw)
- net at J24.1 (Pin_1): now also SW13.2 (B), C10.1
- net at J24.3 (Pin_3): now also R3.1
- net +5V: now reaches SW13.1 (A)
- net +5V: now also C10.1, C10.1, D1.2 (A), L2.2, R3.1
- net USART_{3}_TX: now reaches U1.47 (PB10)
- net USART_{3}_RX: now reaches U1.48 (PB11)
- net SClk_{3}: now reaches U1.89 (PB3)
- net MISO_{3}: now reaches U1.90 (PB4)
- net MOSI_{3}: now reaches U1.91 (PB5)
- net VBUS: no longer names the net of J1.A4 (VBUS), J1.A9 (VBUS), J1.B4 (VBUS), J1.B9 (VBUS)
- new net: R3.1, R3.2, U11.4 (En)
- new net: C10.2, L2.1, R3.1, U8.11 (Sw), U8.12 (Sw)
- new net: C10.2, C10.2, R3.2 (x2)
- new net: C10.1, U8.10 (Bst)
- new net: C10.1, R3.1, R3.2, U8.8 (FB)
- new net: D1.1 (K), R3.2 (x2)
- new net: R3.1, U11.5 (ROn)
- new net: C10.2, U11.7 (FPWM), U11.9 (V_{CC})
- new net: R3.2, U14.1
- new net: C10.1, R3.1, R3.2, U11.8 (FB)
- new net: R3.1, U14.4
- new net: C10.2, U8.6 (SS)
- new net: C10.1, U11.10 (Bst)
- new net: C10.2, U11.6 (SS)
- new net: R3.1, R3.2, U8.4 (En)
- new net: R3.1, U8.5 (ROn)
- new net: C10.2, U8.7 (FPWM), U8.9 (V_{CC})
- new net Bed: U9.14 (D)
- new net Fan0: U9.3 (A)
- new net Fan1: U9.6 (B)
- new net Fan2: U12.3 (A)
- new net Fan3: U12.6 (B)
- new net Fan4: U13.3 (A)
- new net Fan5: U13.6 (B)
- new net HE0: U12.14 (D)
- new net HE1: U12.10 (C)
- new net HE2: U13.14 (D)
- new net HE3: U13.10 (C)
- new net Probe: R3.1, U14.3
- no-connect marks 8 -> 9
Other:
- note removed: "24→12V Step-Down"
- note removed: "I spend good f*cking money on this IC so y'all better use it"
- moved on the sheet: D1, F2, F3, F4, F5, J10, J11, J22, J24, Q1A, Q1B, R3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

Commit message: nearing first prototype woot! copyediting over entire board, fixed some mistakes
Parts:
- removed J22: SPI-something, Connector_IDC:IDC-Header_2x05_P2.54mm_Vertical, symbol Connector_Generic:Conn_02x05_Odd_Even
- added C10 (x2): 10μF, AlphaLib:0603C, symbol Device:C_Small
- added C10 (x3): 220nF, AlphaLib:0402C, symbol Device:C_Small
- added C10 (x2): 2.2μF, AlphaLib:0402C, symbol Device:C_Small
- added U15: AMS1117-3.3, Package_TO_SOT_SMD:SOT-223-3_TabPin2, symbol Regulator_Linear:AMS1117-3.3
- C10: value 1μF -> 1μF 50V
- C10: value 100nF -> 100nF 50V
- R3: value 50kΩ -> 51kΩ
Connections:
- net USART_{1}_TX is gone; now on net _{M4}Step: U1.68 (PA9)
- net +3.3V: now also U1.21 (VREF+), C10.1, C10.1, C10.1, C10.1, U15.2 (VO)
- net +5V: now also J10.10 (Pin_10), J11.10 (Pin_10), C10.1, U15.3 (VI)
- net Bed: now also U1.36 (PB1)
- net ES0: now also U1.23 (PA0)
- net ES1: now also U1.24 (PA1)
- net ES2: now also U1.25 (PA2)
- net ES3: now also U1.26 (PA3)
- net Fan0: now also U1.41 (PE10)
- net Fan1: now also U1.42 (PE11)
- net Fan2: now also U1.43 (PE12)
- net Fan3: now also U1.44 (PE13)
- net Fan4: now also U1.45 (PE14)
- net Fan5: now also U1.46 (PE15)
- net GND: now also J10.9 (Pin_9), J11.9 (Pin_9), C10.2, C10.2, C10.2, C10.2, C10.2, C10.2, C10.2, U15.1 (GND)
- net HE0: now also U1.37 (PB2)
- net HE1: now also U1.38 (PE7)
- net HE2: now also U1.39 (PE8)
- net HE3: now also U1.40 (PE9)
- net MISO_{3}: now also J11.1 (Pin_1)
- net MOSI_{3}: now also J11.6 (Pin_6)
- net Probe: now also U1.72 (PA13)
- net SClk_{3}: now also J11.2 (Pin_2)
- net _{M10}Dir: now also U1.82 (PD1)
- net _{M10}Step: now also U1.81 (PD0)
- net _{M12}Dir: now also U1.86 (PD5)
- net _{M12}Step: now also U1.85 (PD4)
- net _{M20}Dir: now also U1.3 (PE4)
- net _{M20}Step: now also U1.2 (PE3)
- net _{M22}Dir: now also U1.7 (PC13)
- net _{M22}Step: now also U1.5 (PE6)
- net _{M4}Dir: now also U1.67 (PA8)
- net _{M5}Dir: now also U1.78 (PC10)
- net _{M5}Step: now also U1.79 (PC11)
- net ~{Reset}: now also J11.8 (Pin_8)
- net Btn_En2: now reaches J11.3 (Pin_3)
- net Btn_En2: now also U1.60 (PD13)
- net SD_CS: now reaches J11.4 (Pin_4)
- net SD_CS: now also U1.57 (PD10)
- net Btn_En1: now reaches J11.5 (Pin_5)
- net Btn_En1: now also U1.56 (PD9)
- net SD_Det: now reaches J11.7 (Pin_7)
- net SD_Det: now also U1.55 (PD8)
- net Buzzer: now reaches J10.1 (Pin_1)
- net Buzzer: now also U1.62 (PD15)
- net Btn_Enc: now reaches J10.2 (Pin_2)
- net Btn_Enc: now also U1.61 (PD14)
- net LCD_En: now reaches J10.3 (Pin_3)
- net LCD_En: now also U1.58 (PD11)
- net LCD_Rs: now reaches J10.4 (Pin_4)
- net LCD_Rs: now also U1.59 (PD12)
- net LCD_D4: now reaches J10.5 (Pin_5)
- net LCD_D4: now also U1.54 (PB15)
- net LCD_D5: now reaches J10.6 (Pin_6)
- net LCD_D5: now also U1.53 (PB14)
- net LCD_D6: now reaches J10.7 (Pin_7)
- net LCD_D6: now also U1.52 (PB13)
- net LCD_D7: now reaches J10.8 (Pin_8)
- net LCD_D7: now also U1.51 (PB12)
- net _{M20}~{En}: now reaches U1.1 (PE2)
- net _{M3}~{En}: now reaches U1.29 (PA4)
- net _{M4}Diag1: now reaches U1.33 (PC4)
- net _{M1}~{En}: now reaches U1.34 (PC5)
- net _{M1}Dir: now reaches U1.35 (PB0)
- net _{M20}~{CS}: now reaches U1.4 (PE5)
- net at U1.49 (VCAP_1): now also C10.1
- net _{M0}~{En}: now reaches U1.63 (PC6)
- net _{M0}UART: now reaches U1.64 (PC7)
- net _{M0}Step: now reaches U1.65 (PC8)
- net _{M0}Dir: now reaches U1.66 (PC9)
- net at U1.73 (VCAP_2): now also C10.1
- net _{M4}~{CS}: now reaches U1.76 (PA14)
- net _{M5}~{En}: now reaches U1.77 (PA15)
- net _{M22}~{En}: now reaches U1.8 (PC14)
- net _{M5}~{CS}: now reaches U1.80 (PC12)
- net _{M10}~{En}: now reaches U1.83 (PD2)
- net _{M10}~{CS}: now reaches U1.84 (PD3)
- net _{M12}~{En}: now reaches U1.87 (PD6)
- net _{M12}~{CS}: now reaches U1.88 (PD7)
- net _{M22}~{CS}: now reaches U1.9 (PC15)
- net _{M1}Step: now reaches U1.92 (PB6)
- net _{M1}UART: now reaches U1.93 (PB7)
- net _{M2}Dir: now reaches U1.95 (PB8)
- net _{M2}Step: now reaches U1.96 (PB9)
- net _{M2}UART: now reaches U1.97 (PE0)
- net _{M2}~{En}: now reaches U1.98 (PE1)
- net MISO_{1} renamed _{M3}Step
- net MOSI_{1} renamed _{M3}Dir
- net SClk_{1} renamed _{M3}UART
- net USART_{1}_RX renamed _{M4}~{En}
Other:
- note removed: "8 pin LDO FPC connector"
- note removed: "ALLOCATE PINS MOSI1 MISO1 SCLK1 14x4 Motor Control (56 I/O) Fan (6 PWM) Thermistor (6 ADC)"
- note removed: "Most pins on STM32 tolerate 5V logic (VDD+4.0 max, <5.2 recommended) https://www.st.com/resource/en/datasheet/stm32f446mc.pdf"
- note removed: "RPi Zero --USB--> USB-A (Camera) / / / USB-C /---UART----> MCU"
- moved on the sheet: C10, D1, F1, F2, F3, F4, F5, F6, FID1, FID2, FID3, FID4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

Commit message: test new gitignore with completed mainboard
Parts:
- R3: value kΩ -> 100kΩ
Changed lines of the file:
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@@
       (effects (font (size 0.8 0.8)) (justify right))
     )
-    (property "Value" "kΩ" (at 153.67 73.66 90)
+    (property "Value" "100kΩ" (at 153.67 73.66 90)
       (effects (font (size 0.6 0.6)))
     )
