File: hardware/mainboard/mainboard.kicad_sch (KiCad schematic)
At the start: 79 parts, among them J1 USB 2.0, J10 JST XH, J11 JST XH, J12 EXP1, J13 EXP2, J2 JST XH, J3 Power In, J4 JST XH, J5 JST XH, J6 JST XH, J7 JST XH, J8 JST XH, J9 JST XH, Q1 AGM308MBP, SW1 SW_SPDT, SW2 SW_SPDT, SW9 SW_SPDT, U1 STM32F407ZETx, U2 CD40109B, U3 CD40109B, U4 CD40109B, U5 LTV-357T, U6 AMS1117-3.3, Y1 12 MHz

Commit message: tested SMD style XH connectors — didn't work very well alas
Parts:
- removed C10 (x3): 1μF, AlphaLib:0402C, symbol Device:C_Small
- removed J12: EXP1, corevus:IDC-Header_2x05_P2.54mm_Vertical_SMD, symbol Connector_Generic:Conn_02x05_Odd_Even
- removed J7: JST XH, Connector_JST:JST_XH_B3B-XH-A_1x03_P2.50mm_Vertical, symbol Connector:Conn_01x03_Pin
- removed R3 (x3): 4.7kΩ, AlphaLib:0402R, symbol Device:R_Small
- removed R3: 10kΩ, AlphaLib:0402R, symbol Device:R_Small
- added C10 (x5): 1μF, AlphaLib:0402C, symbol Device:C_Small
- added D1 (x10): Red, AlphaLib:0402LED, symbol Device:LED_Small
- added D27, D29, D33, D34, D35, D4: sth, symbol Device:D_Small
- added D3: sth, symbol Device:D_Schottky_Small
- added FB1: GZsth, AlphaLib:0603, symbol Device:FerriteBead_Small
- added H5: Back, corevus:M3_M2.5_PCB_Nut, symbol Mechanical:MountingHole
- added J12, J14, J15, J16, J17, J18, J19, J7: JST XH, corevus:ShouHan_2.54-2PLT, symbol Connector:Conn_01x02_Pin
- added J28: EXP2, corevus:IDC-Header_2x05_P2.54mm_Vertical_SMD, symbol Connector_Generic:Conn_02x05_Odd_Even
- added J29, J30, J31: 2x3p, corevus:HCTL_PinHeader_2x03_SMD, symbol Connector_Generic:Conn_02x03_Odd_Even
- added J32, J33, J34: XH, corevus:ShouHan_2.54-3PLT, symbol Connector:Conn_01x03_Pin
- added NT1, NT2: NetTie_2, corevus:NetTie-2_SMD_Pad0.1mm, symbol Device:NetTie_2
- added Q20, Q21, Q22, Q28, Q29, Q30: AO3400, Package_TO_SOT_SMD:SOT-23, symbol Device:Q_NMOS_GSD
- added R3 (x23): 4.7kΩ, AlphaLib:0402R, symbol Device:R_Small
- added R3 (x10): 10kΩ, AlphaLib:0402R, symbol Device:R_Small
- added R3 (x6): 100Ω, AlphaLib:0402R, symbol Device:R_Small
- added R3 (x3): 200Ω, AlphaLib:0402R, symbol Device:R_Small
- added R3: 1kΩ, AlphaLib:0402R, symbol Device:R_Small
- added SW3: SW_Push, corevus:XKB_TS-1187A, symbol Switch:SW_Push
- C10: value 20pF -> 15pF
- J10, J11, J8, J9: footprint Connector_JST:JST_XH_B2B-XH-A_1x02_P2.50mm_Vertical -> corevus:ShouHan_2.54-2PLT
- J13: value EXP2 -> EXP1
- J4, J5, J6: value JST XH -> XH; footprint Connector_JST:JST_XH_B3B-XH-A_1x03_P2.50mm_Vertical -> corevus:ShouHan_2.54-3PLT
- R3: value 330Ω -> 1kΩ
- renumbered Q1 to Q4
Connections:
- net Th_{2} is gone; now on net VSSA: J10.1 (Pin_1)
- net Th_{3} is gone; now on net VSSA: J11.1 (Pin_1)
- net +24V: now also D27.1 (K), D29.1 (K), D33.1 (K), D34.1 (K), D35.1 (K), D4.1 (K), J14.1 (Pin_1), J15.1 (Pin_1), J16.1 (Pin_1), J17.1 (Pin_1), J18.1 (Pin_1), J19.1 (Pin_1)
- net +3.3V: now also J4.3 (Pin_3), J5.3 (Pin_3), J6.3 (Pin_3), FB1.1, R3.2, R3.2, R3.2, R3.2, R3.2, R3.2, R3.2; no longer J4.1 (Pin_1), J5.1 (Pin_1), J6.1 (Pin_1), R3.2, U1.32 (VREF+), U1.33 (VDDA)
- net +5V: now also D3.1 (K), J28.10 (Pin_10)
- net BG: now also R3.1
- net Bed: now also R3.1
- net Btn_En1: now also J28.5 (Pin_5); no longer J13.5 (Pin_5)
- net Btn_En2: now also J28.3 (Pin_3); no longer J13.3 (Pin_3)
- net Btn_Enc: now also J13.2 (Pin_2)
- net Buzzer: now also J13.1 (Pin_1)
- net ES0: now also J4.1 (Pin_1), D1.1 (K), R3.1; no longer J4.3 (Pin_3)
- net ES1: now also J5.1 (Pin_1), D1.1 (K), R3.1; no longer J6.3 (Pin_3)
- net ES2: now also J6.1 (Pin_1), D1.1 (K), R3.1; no longer J5.3 (Pin_3)
- net Fan0: now also R3.1
- net Fan1: now also R3.1
- net Fan2: now also R3.1
- net Fan3: now also R3.1
- net Fan4: now also R3.1
- net Fan5: now also R3.1
- net GND: now also SW9.3 (C), J28.9 (Pin_9), NT1.1, Q20.2 (S), Q21.2 (S), Q22.2 (S), Q28.2 (S), Q29.2 (S), Q30.2 (S), R3.1, R3.1, R3.1, R3.1, R3.1, R3.1, R3.1, R3.2, R3.2, R3.2, R3.2, R3.2, R3.2, R3.2, R3.2, R3.2, R3.2, R3.2, R3.2, R3.2, R3.2, R3.2, R3.2, R3.2, R3.2; no longer C10.1, J10.2 (Pin_2), J11.2 (Pin_2), J8.2 (Pin_2), J9.2 (Pin_2), U1.31 (VSSA)
- net HE0: now also R3.1
- net HE1: now also R3.1
- net HE2: now also R3.1
- net HE3: now also R3.1
- net HeEn: now also SW9.2 (B), D1.2 (A)
- net LCD_D4: now also J13.5 (Pin_5)
- net LCD_D5: now also J13.6 (Pin_6)
- net LCD_D6: now also J13.7 (Pin_7)
- net LCD_D7: now also J13.8 (Pin_8)
- net LCD_En: now also J13.3 (Pin_3)
- net LCD_Rs: now also J13.4 (Pin_4)
- net MISO_{3}: now also J28.1 (Pin_1); no longer J13.1 (Pin_1)
- net MOSI_{3}: now also J28.6 (Pin_6); no longer J13.6 (Pin_6)
- net SClk_{3}: now also J28.2 (Pin_2); no longer J13.2 (Pin_2)
- net SD_CS: now also J28.4 (Pin_4); no longer J13.4 (Pin_4)
- net SD_Det: now also J28.7 (Pin_7); no longer J13.7 (Pin_7)
- net ~{Reset}: now also J28.8 (Pin_8); no longer J13.8 (Pin_8)
- net at SW9.1 (A): now also R3.1
- net at J1.A4 (VBUS), J1.A9 (VBUS), J1.B4 (VBUS)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: now also D3.2 (A)
- net T0: now reaches U1.26 (PC0)
- net T0: now also C10.2, J8.2 (Pin_2), R3.1
- net T1: now reaches U1.27 (PC1)
- net T1: now also C10.2, J7.2 (Pin_2), R3.1
- net T2: now reaches U1.28 (PC2)
- net T2: now also J9.2 (Pin_2), C10.2, R3.1
- net T3: now reaches U1.29 (PC3)
- net T3: now also J10.2 (Pin_2), C10.2, R3.1
- net T4: now reaches U1.34 (PA0)
- net T4: now also J11.2 (Pin_2), C10.2, R3.1
- net T5: now reaches U1.35 (PA1)
- net T5: now also C10.2, J12.2 (Pin_2), R3.1
- net USART2_TX: now reaches U1.36 (PA2)
- net USART2_RX: now reaches U1.37 (PA3)
- net SPI1_SCK: now reaches U1.41 (PA5)
- net SPI1_MISO: now reaches U1.42 (PA6)
- net SPI1_MOSI: now reaches U1.43 (PA7)
- removed net Th_{0}: C10.2, J8.1 (Pin_1), R3.1
- net Th_{1} renamed VSSA
- net VSSA: now also C10.1, J8.1 (Pin_1), U1.31 (VSSA), C10.1, C10.1, C10.1, C10.1, C10.1, J12.1 (Pin_1), J7.1 (Pin_1), NT1.2
- new net: D1.1 (K), R3.1 (x6)
- new net: D1.2 (A), R3.1, R3.2 (x6)
- new net: Q30.1 (G), R3.2
- new net: D34.2 (A), J18.2 (Pin_2), Q29.3 (D)
- new net: D27.2 (A), J15.2 (Pin_2), Q21.3 (D)
- new net: D1.1 (K), R3.2
- new net: NT2.2, U1.32 (VREF+)
- new net: D35.2 (A), J19.2 (Pin_2), Q30.3 (D)
- new net: D29.2 (A), J16.2 (Pin_2), Q22.3 (D)
- new net: D1.2 (A), R3.1 (x3)
- new net: D4.2 (A), J14.2 (Pin_2), Q20.3 (D)
- new net: D33.2 (A), J17.2 (Pin_2), Q28.3 (D)
- new net: Q29.1 (G), R3.2
- new net: Q20.1 (G), R3.2
- new net: Q21.1 (G), R3.2
- new net: Q22.1 (G), R3.2
- new net: Q28.1 (G), R3.2
- new net VDDA: FB1.2, NT2.1, R3.2, R3.2, R3.2, R3.2, R3.2, R3.2, U1.33 (VDDA)
- no-connect marks 9 -> 8
Other:
- removed sheet Fans 0, 1
- removed sheet Fans 2, 3
- removed sheet Fans 4, 5
- moved on the sheet: C10, D1, J1, J8, R3, SW1, SW9, U2, U3, U4

Commit message: fan ports
Parts:
- removed C15: 220μF 35V, Capacitor_SMD:CP_Elec_8x10.5, symbol Device:C_Polarized_Small_US
- removed D1 (x5): Red, AlphaLib:0402LED, symbol Device:LED_Small
- removed D29, D33, D34, D35: sth, symbol Device:D_Small
- removed J15: JST XH, corevus:ShouHan_2.54-2PLT, symbol Connector:Conn_01x02_Pin
- removed J32, J33, J34: XH, corevus:ShouHan_2.54-3PLT, symbol Connector:Conn_01x03_Pin
- removed Q4 (x3): AGM308MBP, corevus:AGM308MBP, symbol Device:Q_Dual_NMOS_S1G1S2G2D2D2D1D1
- removed R3 (x5): 4.7kΩ, AlphaLib:0402R, symbol Device:R_Small
- removed R3 (x10): 10kΩ, AlphaLib:0402R, symbol Device:R_Small
- removed R3 (x6): 100Ω, AlphaLib:0402R, symbol Device:R_Small
- added C10 (x14): 100nF, AlphaLib:0402C, symbol Device:C_Small
- added D1 (x11): Red, AlphaLib:0402LED, symbol Device:LED_Small
- added D30, D31, D36, D37, D38, D39, D41, D43, D45, D47: 1N4148, corevus:D_SOD-323, symbol Device:D_Small
- added J15: XH, corevus:JST_XH_1x03, symbol Connector:Conn_01x03_Pin
- added J32, J33, J34, J35: JST XH, corevus:JST_XH_1x02, symbol Connector:Conn_01x02_Pin
- added J36, J37: JST XH, corevus:JST_XH_1x03, symbol Connector:Conn_01x03_Pin
- added J38: JST XH, corevus:JST_XH_1x04, symbol Connector:Conn_01x04_Pin
- added Q26 (x2): 60N03F, corevus:MOSFET_DFN8, symbol corevus:Q_NMOS-E_Generic_SSSGDDDD
- added Q27, Q3, Q31, Q32, Q33: AO3400, Package_TO_SOT_SMD:SOT-23, symbol Device:Q_NMOS_GSD
- added R3 (x10): 4.7kΩ, AlphaLib:0402R, symbol Device:R_Small
- added R3: 200Ω, AlphaLib:0402R, symbol Device:R_Small
- added R3: 10kΩ, AlphaLib:0402R, symbol Device:R_Small
- C12: value 220μF 35V -> 470μF 63V; footprint Capacitor_SMD:CP_Elec_8x10.5 -> Capacitor_THT:CP_Radial_D12.5mm_P5.00mm
- D27, D4: value sth -> 1N4148; footprint (none) -> corevus:D_SOD-323
- D3: value sth -> SS54; footprint (none) -> Diode_SMD:D_SMA
- J10, J11, J12, J14, J16, J17, J18, J19, J7, J8, J9: footprint corevus:ShouHan_2.54-2PLT -> corevus:JST_XH_1x02
- J2: footprint Connector_JST:JST_XH_B3B-XH-A_1x03_P2.50mm_Vertical -> corevus:JST_XH_1x03
- J4, J5, J6: footprint corevus:ShouHan_2.54-3PLT -> corevus:JST_XH_1x03
- SW3: value SW_Push -> SPST
Connections:
- net ES0 is gone; now on net E0: D1.1 (K), J4.1 (Pin_1)
- net ES1 is gone; now on net E1: D1.1 (K), J5.1 (Pin_1)
- net ES2 is gone; now on net E2: D1.1 (K), J6.1 (Pin_1)
- net +24V: now also D30.1 (K), D31.1 (K), D36.1 (K), D37.1 (K), D38.1 (K), D39.1 (K), D41.1 (K), D43.1 (K), D45.1 (K), D47.1 (K), J32.1 (Pin_1), J33.1 (Pin_1), J34.1 (Pin_1), J35.1 (Pin_1), J36.1 (Pin_1), J37.1 (Pin_1), J38.1 (Pin_1)
- net +3.3V: now also U1.143 (PDR_ON), C10.1, C10.1, C10.1, C10.1, C10.1, C10.1, C10.1, C10.1, C10.1, C10.1, C10.1, C10.1, C10.1, J15.3 (Pin_3), R3.1, R3.2
- net BG: now also Q26.4 (G), Q26.4 (G)
- net Bed_H-: now also Q26.5 (D), Q26.5 (D), Q26.6 (D), Q26.6 (D), Q26.7 (D), Q26.7 (D), Q26.8 (D), Q26.8 (D)
- net GND: now also SW3.1, C10.2, C10.2, C10.2, C10.2, C10.2, C10.2, C10.2, C10.2, C10.2, C10.2, C10.2, C10.2, C10.2, C10.2, J15.2 (Pin_2), Q26.1 (S), Q26.1 (S), Q26.2 (S), Q26.2 (S), Q26.3 (S), Q26.3 (S), Q27.2 (S), Q3.2 (S), Q31.2 (S), Q32.2 (S), Q33.2 (S), R3.2, R3.2, R3.2, R3.2, R3.2, R3.2, R3.2, R3.2, R3.2, R3.2
- net _{M0}Dir: now also U1.113 (PC12)
- net _{M0}Step: now also U1.114 (PD0)
- net _{M0}UART: now also U1.115 (PD1)
- net _{M0}~{En}: now also U1.112 (PC11)
- net _{M10}Dir: now also U1.2 (PE3)
- net _{M10}Step: now also U1.1 (PE2)
- net _{M10}~{CS}: now also U1.4 (PE5)
- net _{M10}~{En}: now also U1.3 (PE4)
- net _{M12}Dir: now also U1.7 (PC13)
- net _{M12}Step: now also U1.5 (PE6)
- net _{M12}~{CS}: now also U1.9 (PC15)
- net _{M12}~{En}: now also U1.8 (PC14)
- net _{M1}Dir: now also U1.117 (PD3)
- net _{M1}Step: now also U1.118 (PD4)
- net _{M1}UART: now also U1.119 (PD5)
- net _{M1}~{En}: now also U1.116 (PD2)
- net _{M20}Dir: now also U1.11 (PF1)
- net _{M20}Step: now also U1.10 (PF0)
- net _{M20}~{CS}: now also U1.13 (PF3)
- net _{M20}~{En}: now also U1.12 (PF2)
- net _{M22}Dir: now also U1.15 (PF5)
- net _{M22}Step: now also U1.14 (PF4)
- net _{M22}~{CS}: now also U1.19 (PF7)
- net _{M22}~{En}: now also U1.18 (PF6)
- net _{M2}Dir: now also U1.123 (PD7)
- net _{M2}Step: now also U1.124 (PG9)
- net _{M2}UART: now also U1.125 (PG10)
- net _{M2}~{En}: now also U1.122 (PD6)
- net _{M3}Dir: now also U1.127 (PG12)
- net _{M3}Step: now also U1.128 (PG13)
- net _{M3}UART: now also U1.129 (PG14)
- net _{M3}~{En}: now also U1.126 (PG11)
- net _{M4}Diag1: now also U1.140 (PB9)
- net _{M4}Dir: now also U1.142 (PE1)
- net _{M4}Step: now also U1.139 (PB8)
- net _{M4}~{CS}: now also U1.137 (PB7)
- net _{M4}~{En}: now also U1.141 (PE0)
- net _{M5}Dir: now also U1.134 (PB4)
- net _{M5}Step: now also U1.133 (PB3)
- net _{M5}~{CS}: now also U1.132 (PG15)
- net _{M5}~{En}: now also U1.135 (PB5)
- net F6_Gate: now reaches Q30.1 (G)
- net F6_Gate: now also D1.2 (A)
- net at J18.2 (Pin_2): now also D31.2 (A), Q27.3 (D); no longer Q29.3 (D)
- net at D27.2 (A), Q21.3 (D): now also J16.2 (Pin_2)
- net F0_Gate: now reaches D1.2 (A)
- net F0_Gate: now also Q20.1 (G)
- net at Q30.3 (D): now also D38.2 (A), J33.2 (Pin_2); no longer J19.2 (Pin_2)
- net at Q22.3 (D): now also J17.2 (Pin_2), D30.2 (A); no longer J16.2 (Pin_2)
- net at Q28.3 (D): now also J19.2 (Pin_2), D36.2 (A); no longer J17.2 (Pin_2)
- net F5_Gate: now reaches Q29.1 (G)
- net F5_Gate: now also D1.2 (A)
- net F1_Gate: now reaches Q21.1 (G)
- net F1_Gate: now also D1.2 (A)
- net F2_Gate: now reaches Q22.1 (G)
- net F2_Gate: now also D1.2 (A)
- net _{M5}Diag1: now reaches U1.136 (PB6)
- net E1: now reaches U1.20 (PF8)
- net E2: now reaches U1.21 (PF9)
- net E3: now reaches U1.22 (PF10)
- net E3: now also D1.1 (K), J15.1 (Pin_1)
- net at U1.25 (NRST): now also SW3.2, C10.1, R3.2
- net E0: now reaches U1.40 (PA4)
- net F4_Gate: now reaches Q28.1 (G)
- net F4_Gate: now also D1.2 (A)
- new net: D39.2 (A), J34.2 (Pin_2), Q31.3 (D)
- new net: D1.1 (K), R3.1 (x10)
- new net: D45.2 (A), J37.2 (Pin_2), Q33.3 (D)
- new net: D1.2 (A), R3.1
- new net: D37.2 (A), J32.2 (Pin_2), Q29.3 (D)
- new net: D47.2 (A), J38.2 (Pin_2)
- new net: D41.2 (A), J35.2 (Pin_2), Q32.3 (D)
- new net: D43.2 (A), J36.2 (Pin_2), Q3.3 (D)
- new net F10_Gate: D1.2 (A), Q33.1 (G)
- new net F11: J38.4 (Pin_4)
- new net F11_FG: J38.3 (Pin_3)
- new net F3_Gate: D1.2 (A), Q27.1 (G)
- new net F7_Gate: D1.2 (A), Q31.1 (G)
- new net F8_Gate: D1.2 (A), Q32.1 (G)
- new net F9_Gate: D1.2 (A), Q3.1 (G)
Other:
- note removed: "3x2 7mΩ FETs dissipate ~50 mW at 8A."
- moved on the sheet: D1, D4, J14, Q20, R3, SW1, SW3

Commit message: this is immediately before i switch the terminus USB hub with the corechips
Parts:
- removed D1 (x2): Red, AlphaLib:0402LED, symbol Device:LED_Small
- removed D43, D45, D47: 1N4148, corevus:D_SOD-323, symbol Device:D_Small
- removed J14, J16: JST XH, corevus:JST_XH_1x02, symbol Connector:Conn_01x02_Pin
- removed J29, J30, J31: 2x3p, corevus:HCTL_PinHeader_2x03_SMD, symbol Connector_Generic:Conn_02x03_Odd_Even
- removed J36, J37: JST XH, corevus:JST_XH_1x03, symbol Connector:Conn_01x03_Pin
- removed J38: JST XH, corevus:JST_XH_1x04, symbol Connector:Conn_01x04_Pin
- removed Q20, Q21, Q3, Q33: AO3400, Package_TO_SOT_SMD:SOT-23, symbol Device:Q_NMOS_GSD
- removed R3 (x3): 4.7kΩ, AlphaLib:0402R, symbol Device:R_Small
- removed U5: LTV-357T, Package_SO:SO-4_4.4x3.6mm_P2.54mm, symbol Isolator:LTV-357T
- added C10 (x2): 100nF, AlphaLib:0402C, symbol Device:C_Small
- added C13 (x3): 10μF 50V, Capacitor_SMD:C_1206_3216Metric, symbol Device:C_Small
- added C13 (x4): 22μF 25V, Capacitor_SMD:C_1206_3216Metric, symbol Device:C_Small
- added C13 (x2): 2.2μF, AlphaLib:0402C, symbol Device:C_Small
- added D1: Red, AlphaLib:0402LED, symbol Device:LED_Small
- added D46, D48: 1N4148, corevus:D_SOD-323, symbol Device:D_Small
- added J14, J16: JST XH, corevus:JST_XH_1x04, symbol Connector:Conn_01x04_Pin
- added J36: Conn_02x09_Odd_Even, Connector_PinSocket_2.54mm:PinSocket_2x09_P2.54mm_Vertical, symbol Connector_Generic:Conn_02x09_Odd_Even
- added L1, L2: 10μH, corevus:CJiang_FXL1040, symbol Device:L
- added OC1: PC3H7, Package_SO:SOP-4_4.4x2.6mm_P1.27mm, symbol PCM_Optocoupler_AKL:PC3H7
- added Q26 (x4): 60N03F, corevus:MOSFET_DFN8, symbol corevus:Q_NMOS-E_Generic_SSSGDDDD
- added R3: 4.7kΩ, AlphaLib:0402R, symbol Device:R_Small
- added R3 (x2): 330Ω, AlphaLib:0402R, symbol Device:R_Small
- added R3: 1.8kΩ, AlphaLib:0402R, symbol Device:R_Small
- added R3: 1kΩ, AlphaLib:0402R, symbol Device:R_Small
- added U14: CD4504B, Package_SO:SOP-16_3.9x9.9mm_P1.27mm, symbol 4xxx:4504
- added U15, U5: RT8110B, Package_TO_SOT_SMD:TSOT-23-8, symbol corevus:RT8110B
- C12, C13, C14, C16, C17: footprint Capacitor_THT:CP_Radial_D12.5mm_P5.00mm -> corevus:CP_Radial_D12.5mm_P5.00mm
- J13, J28: footprint corevus:IDC-Header_2x05_P2.54mm_Vertical_SMD -> Connector_IDC:IDC-Header_2x05_P2.54mm_Vertical
Connections:
- net +48V is gone; now on net VMB: R3.1
- net +12V: now also SW9.1 (A), C13.1, C13.1, J36.1 (Pin_1), J36.11 (Pin_11), J36.12 (Pin_12), J36.13 (Pin_13), J36.14 (Pin_14), J36.2 (Pin_2), L1.2, R3.2
- net +24V: now also SW2.1 (A), C13.1, C13.1, C13.1, J36.17 (Pin_17), J36.18 (Pin_18), J36.5 (Pin_5), J36.6 (Pin_6), J36.7 (Pin_7), J36.8 (Pin_8), Q26.5 (D), Q26.5 (D), Q26.6 (D), Q26.6 (D), Q26.7 (D), Q26.7 (D), Q26.8 (D), Q26.8 (D), U15.7 (VIN), U5.7 (VIN); no longer D27.1 (K), D30.1 (K), D31.1 (K), D36.1 (K), D37.1 (K), D38.1 (K), D39.1 (K), D4.1 (K), D41.1 (K), J17.1 (Pin_1), J18.1 (Pin_1), J19.1 (Pin_1), J32.1 (Pin_1), J33.1 (Pin_1), J34.1 (Pin_1), J35.1 (Pin_1), R3.1, SW2.3 (C)
- net +3.3V: now also U14.1 (VCC)
- net +5V: now also SW2.3 (C), C13.1, C13.1, L2.2, R3.2; no longer SW2.1 (A)
- net GND: now also D27.2 (A), D4.2 (A), C13.2, C13.2, C13.2, C13.2, C13.2, C13.2, C13.2, C13.2, C13.2, D1.1 (K), J14.2 (Pin_2), J16.2 (Pin_2), OC1.2, Q26.1 (S), Q26.1 (S), Q26.2 (S), Q26.2 (S), Q26.3 (S), Q26.3 (S), R3.2, R3.2, U14.8 (VSS), U15.3 (GND), U5.3 (GND)
- net HeEn: no longer D1.2 (A), SW9.2 (B)
- net Probe: now also OC1.3, R3.2
- net VMB: now also C14.1; no longer C16.1
- net VMC: now also C16.1, R3.1; no longer C14.1
- net at R3.2: now also OC1.1
- net at R3.1: now also OC1.4
- net BG renamed HB_Gate
- net HB_Gate: now also U14.15 (Fout); no longer U4.13 (H)
- net F0_Gate renamed F0
- net F0: now also J14.4 (Pin_4)
- net F1_Gate renamed F1
- net F1: now also J16.4 (Pin_4)
- net HE0_Gate: no longer names the net of U3.13 (H)
- net HE1_Gate: no longer names the net of U3.11 (G)
- net HE2_Gate: no longer names the net of U2.13 (H)
- net HE3_Gate: no longer names the net of U2.11 (G)
- new net: C10.1, D46.1 (K), U15.5 (BOOT)
- new net: C13.1, D46.2 (A), U15.1 (VCC)
- new net: D1.2 (A), SW9.2 (B), U14.16 (VDD)
- new net: C13.1, D48.2 (A), U5.1 (VCC)
- new net: C10.2, L1.1, Q26.1 (S), Q26.2 (S), Q26.3 (S), Q26.5 (D), Q26.6 (D), Q26.7 (D), Q26.8 (D), U15.6 (PHASE)
- new net: Q26.4 (G), U15.4 (UGATE)
- new net: Q26.4 (G), U15.2 (LGATE)
- new net: R3.1, R3.1, U15.8 (FB)
- new net: C10.1, D48.1 (K), U5.5 (BOOT)
- new net: C10.2, L2.1, Q26.1 (S), Q26.2 (S), Q26.3 (S), Q26.5 (D), Q26.6 (D), Q26.7 (D), Q26.8 (D), U5.6 (PHASE)
- new net: Q26.4 (G), U5.2 (LGATE)
- new net: Q26.4 (G), U5.4 (UGATE)
- new net: R3.1, R3.1, U5.8 (FB)
- new net: D1.2 (A), R3.1
- new net F0_FG: J14.3 (Pin_3)
- new net F0_V+: D4.1 (K), J14.1 (Pin_1)
- new net F1_FG: J16.3 (Pin_3)
- new net F1_V+: D27.1 (K), J16.1 (Pin_1)
- new net F2_V+: D30.1 (K), J17.1 (Pin_1)
- new net F3_V+: D31.1 (K), J18.1 (Pin_1), J36.9 (Pin_9)
- new net F4_V+: D36.1 (K), J19.1 (Pin_1), J36.16 (Pin_16)
- new net F5_V+: D37.1 (K), J32.1 (Pin_1), J36.15 (Pin_15)
- new net F6_V+: D38.1 (K), J33.1 (Pin_1)
- new net F7_V+: D39.1 (K), J34.1 (Pin_1)
- new net F8_V+: D41.1 (K), J35.1 (Pin_1)
- new net H0: U14.11 (Ein)
- new net H0_Gate: U14.12 (Eout)
- new net H1: U14.3 (Ain)
- new net H1_Gate: U14.2 (Aout)
- new net H2: U14.5 (Bin)
- new net H2_Gate: U14.4 (Bout)
- new net H3: U14.7 (Cin)
- new net H3_Gate: U14.6 (Cout)
- new net HB: U14.14 (Fin)
Other:
- note added: "0.8V"
- note added: "12.2V"
- note added: "5.16V"
- moved on the sheet: C10, D1, D31, D36, D37, D38, D39, D41, J13, J18, J19, J28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

Commit message: v0.2 feature complete
Parts:
- removed D27, D4: 1N4148, corevus:D_SOD-323, symbol Device:D_Small
- removed R3 (x11): 4.7kΩ, AlphaLib:0402R, symbol Device:R_Small
- removed U2, U3, U4: CD40109B, Package_SO:TSSOP-16_4.4x5mm_P0.65mm, symbol corevus:CD40109B
- added R3 (x5): 10kΩ, AlphaLib:0402R, symbol Device:R_Small
- C10: now not fitted; now left out of the parts list
- C13: value 22μF 25V -> 22μF 10V
- D46, D48: value 1N4148 -> 1N5819
Connections:
- net F6_V+ is gone; now on net +24V: D38.1 (K), J33.1 (Pin_1)
- net F7_V+ is gone; now on net +24V: D39.1 (K), J34.1 (Pin_1)
- net F8_V+ is gone; now on net +24V: D41.1 (K), J35.1 (Pin_1)
- net MISO_{3} is gone; now on net SPI2_MISO: J28.1 (Pin_1)
- net MOSI_{3} is gone; now on net SPI2_MOSI: J28.6 (Pin_6)
- net SClk_{3} is gone; now on net SPI2_SCK: J28.2 (Pin_2)
- net Btn_En1: now also U1.91 (PG6)
- net Btn_En2: now also U1.92 (PG7)
- net Btn_Enc: now also U1.89 (PG4)
- net Buzzer: now also U1.90 (PG5)
- net F0: now also U1.56 (PG0)
- net F0_FG: now also U1.57 (PG1)
- net F0_V+: now also J36.3 (Pin_3)
- net F1: now also U1.58 (PE7)
- net F1_FG: now also U1.59 (PE8)
- net F1_V+: now also J36.4 (Pin_4)
- net F2_Gate: now also U1.60 (PE9)
- net F2_V+: now also J36.9 (Pin_9)
- net F3_Gate: now also U1.63 (PE10)
- net F3_V+: now also J36.10 (Pin_10); no longer J36.9 (Pin_9)
- net F4_Gate: now also U1.64 (PE11)
- net F4_V+: now also J36.15 (Pin_15); no longer J36.16 (Pin_16)
- net F5_Gate: now also U1.65 (PE12)
- net F5_V+: now also J36.16 (Pin_16); no longer J36.15 (Pin_15)
- net F6_Gate: now also U1.66 (PE13)
- net F7_Gate: now also U1.67 (PE14)
- net F8_Gate: now also U1.68 (PE15)
- net GND: now also R3.2, R3.2, R3.2, R3.2, R3.2
- net H0: now also U1.49 (PF11), R3.1
- net H1: now also U1.55 (PF15), R3.1
- net H2: now also U1.54 (PF14), R3.1
- net H3: now also U1.53 (PF13), R3.1
- net HB: now also U1.50 (PF12), R3.1
- net LCD_D4: now also U1.86 (PD15)
- net LCD_D5: now also U1.85 (PD14)
- net LCD_D6: now also U1.82 (PD13)
- net LCD_D7: now also U1.81 (PD12)
- net LCD_En: now also U1.88 (PG3)
- net SD_CS: now also U1.93 (PG8)
- net SD_Det: now also U1.87 (PG2)
- net SPI2_SCK: now reaches U1.74 (PB13)
- net SPI2_MISO: now reaches U1.75 (PB14)
- net SPI2_MOSI: now reaches U1.76 (PB15)
- no-connect marks 8 -> 6
Other:
- moved on the sheet: C10, R3, Y1

Commit message: added more 3D models and created first few renders
Parts:
- added R3 (x9): 10kΩ, AlphaLib:0402R, symbol Device:R_Small
- added U4: SRV05-4, Package_TO_SOT_SMD:SOT-23-6, symbol Power_Protection:SRV05-4
- FB1: value GZsth -> GZ1608
- J1: footprint Connector_USB:USB_C_Receptacle_XKB_U262-16XN-4BVC11 -> corevus:USB_Type-C_16p
Connections:
- net +5V: now also U4.5 (VP)
- net F0: now also R3.1
- net F1: now also R3.1
- net F2_Gate: now also R3.1
- net F3_Gate: now also R3.1
- net F4_Gate: now also R3.1
- net F5_Gate: now also R3.1
- net F6_Gate: now also R3.1
- net F7_Gate: now also R3.1
- net F8_Gate: now also R3.1
- net GND: now also R3.2, R3.2, R3.2, R3.2, R3.2, R3.2, R3.2, R3.2, R3.2, U4.2 (VN)
- net at J1.A6 (D+), J1.B6 (D+), R3.2: now also U4.3 (IO2)
- net at J1.A7 (D-), J1.B7 (D-), R3.2: now also U4.4 (IO3)
- no-connect marks 6 -> 8
Other:
- note removed: "ADD ESD DIODES"
- moved on the sheet: C10, D1, D30, D31, D36, D37, D38, D39, D41, F1, F2, F3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
