File: hardware/corevus-g/driver-tmc5160-integrated.kicad_sch (KiCad schematic)
At the start: 32 parts, among them M6 Micro-Fit 3.0, Q10 DMT6016LFDF, Q11 DMT6016LFDF, Q4 DMT6016LFDF, Q5 DMT6016LFDF, Q6 DMT6016LFDF, Q7 DMT6016LFDF, Q8 DMT6016LFDF, Q9 DMT6016LFDF, U1 TMC5160A-TA

Commit message: test
Parts:
- removed Q10, Q11, Q4, Q5, Q6, Q7, Q8, Q9: DMT6016LFDF, corevus:DMT6016LFDF, symbol corevus:DMT6016LFDF-7
- added D1: Red, AlphaLib:0402LED, symbol Device:LED_Small
- added Q3, Q4: DMHT6016LFJ, corevus:V-DFN5045-12-Type-B, symbol corevus:DMHT6016LFJ
- added R3: 4.7kΩ, AlphaLib:0402R, symbol Device:R_Small
- added R7 (x8): 10Ω, AlphaLib:0402R, symbol Device:R_Small
- M6: footprint corevus:XKB_X3025WRS-04C -> corevus:JST_XH_1x04-Side
- R3: value 1kΩ -> 4.7kΩ
Connections:
- net Diag1: now also R3.2
- net HA1: now also R7.1
- net HA2: now also R7.1
- net HB1: now also R7.1
- net HB2: now also R7.1
- net LA1: now also R7.1
- net LA2: now also R7.1
- net LB1: now also R7.1
- net LB2: now also R7.1
- net Motor_A1: now also M6.2 (-), Q3.10 (D3/S4), Q3.P3 (D3/S4); no longer M6.3
- net Motor_A2: now also M6.1, Q3.3 (S1/D2), Q3.P2 (S1/D2); no longer M6.4
- net Motor_B1: now also M6.4, Q4.10 (D3/S4), Q4.P3 (D3/S4); no longer M6.1
- net Motor_B2: now also M6.3, Q4.3 (S1/D2), Q4.P2 (S1/D2); no longer M6.2 (-)
- net VM: now also Q3.11 (D1/D4), Q3.2 (D1/D4), Q3.P1 (D1/D4), Q4.11 (D1/D4), Q4.2 (D1/D4), Q4.P1 (D1/D4)
- net Vcc_IO: now also D1.2 (A)
- net at R7.1, R9.1: now also Q4.5 (S2), Q4.6 (S2), Q4.7 (S3), Q4.8 (S3)
- net at R7.1, R9.1: now also Q3.5 (S2), Q3.6 (S2), Q3.7 (S3), Q3.8 (S3)
- new net: Q4.1 (G1), R7.2
- new net: D1.1 (K), R3.1
- new net: Q3.9 (G3), R7.2
- new net: Q3.1 (G1), R7.2
- new net: Q3.12 (G4), R7.2
- new net: Q3.4 (G2), R7.2
- new net: Q4.9 (G3), R7.2
- new net: Q4.12 (G4), R7.2
- new net: Q4.4 (G2), R7.2
Other:
- moved on the sheet: C13, R7, R8, R9
