File: hardware/corevus-g/corevus-g.kicad_sch (KiCad schematic)
At the start: 197 parts, among them J1 USB 2.0, J10 JST XH, J11 JST XH, J12 JST XH, J13 EXP1, J14 JST XH, J15 XH, J16 JST XH, J17 JST XH, J18 JST XH, J19 JST XH, J2 JST XH, J25 1x6, J28 EXP2, J29 1x6, J3 Power In, J30 1x6, J32 JST XH, J33 JST XH, J34 JST XH, J35 JST XH, J4 XH, J5 XH, J6 XH, J7 JST XH, J8 JST XH, J9 JST XH, Q22 AO3400, Q26 60N03F, Q27 AO3400, Q28 AO3400, Q29 AO3400, Q30 AO3400, Q31 AO3400, Q32 AO3400, SW1 SW_SPDT, SW2 SW_SPDT, SW3 SPST, SW9 SW_SPDT, U1 STM32F407ZETx, U14 CD4504B, U15 RT8110B, U4 SRV05-4, U5 RT8110B, U6 AMS1117-3.3, Y1 12 MHz

Commit message: aonteuhasntoidanouidoenuthidntoehuid
Parts:
- Q26: symbol corevus:Q_NMOS-E_Generic_SSSGDDDD -> corevus:NMOS_DFN8
Connections:
- net Bed_H-: no longer Q26.5 (D), Q26.6 (D), Q26.7 (D), Q26.8 (D)
- net GND: now also C10.1; no longer C10.2
- net at U1.106 (VCAP_2): now also C10.2; no longer C10.1
- new net: Q26.5 (D), Q26.6 (D), Q26.7 (D), Q26.8 (D)
Other:
- moved on the sheet: C10, C13, D1, D46, D48, L1, L2, R3, U15, U5

Commit message: version control appears to have magically disappeared the single and dual 2160 driver files :(((((((((, but got some work done on CvG nonetheless
Parts:
- removed C10 (x2): 10μF, AlphaLib:0603C, symbol Device:C_Small
- removed C10 (x2): 100nF, AlphaLib:0402C, symbol Device:C_Small
- removed C10: 100nF 50V, AlphaLib:0402C, symbol Device:C_Small
- removed C13 (x3): 10μF 50V, Capacitor_SMD:C_1206_3216Metric, symbol Device:C_Small
- removed C13 (x2): 22μF 10V, Capacitor_SMD:C_1206_3216Metric, symbol Device:C_Small
- removed C13 (x2): 1μF, AlphaLib:0402C, symbol Device:C_Small
- removed C13 (x2): 22μF 25V, Capacitor_SMD:C_1206_3216Metric, symbol Device:C_Small
- removed D1 (x16): Red, AlphaLib:0402LED, symbol Device:LED_Small
- removed D3: SS54, Diode_SMD:D_SMA, symbol Device:D_Schottky_Small
- removed D30, D31, D36, D37, D38, D39, D41: 1N4148, corevus:D_SOD-323, symbol Device:D_Small
- removed D46, D48: 1N5819, corevus:D_SOD-323, symbol Device:D_Schottky_Small
- removed J15, J4, J5, J6: XH, corevus:JST_XH_1x03, symbol Connector:Conn_01x03_Pin
- removed J16: JST XH, corevus:JST_XH_1x04, symbol Connector:Conn_01x04_Pin
- removed J18, J19, J32, J33, J34, J35: JST XH, corevus:JST_XH_1x02, symbol Connector:Conn_01x02_Pin
- removed J2: JST XH, corevus:JST_XH_1x03, symbol Connector:Conn_01x03_Pin
- removed J25, J29, J30: 1x6, corevus:PinHeader_1x06_P2.54mm_Vertical, symbol Connector:Conn_01x06_Pin
- removed J3: Power In, corevus:DBT50G-9.5-6P, symbol Connector:Screw_Terminal_01x06
- removed OC1: PC3H7, Package_SO:SOP-4_4.4x2.6mm_P1.27mm, symbol PCM_Optocoupler_AKL:PC3H7
- removed Q26 (x6): 60N03F, corevus:MOSFET_DFN8, symbol corevus:NMOS_DFN8
- removed Q27, Q31, Q32: AO3400, Package_TO_SOT_SMD:SOT-23, symbol Device:Q_NMOS_GSD
- removed R3 (x10): 4.7kΩ, AlphaLib:0402R, symbol Device:R_Small
- removed R3 (x15): 10kΩ, AlphaLib:0402R, symbol Device:R_Small
- removed R3 (x4): 1kΩ, AlphaLib:0402R, symbol Device:R_Small
- removed R3 (x4): 470Ω, AlphaLib:0402R, symbol Device:R_Small
- removed R3: 100kΩ, AlphaLib:0402R, symbol Device:R_Small
- removed R3: 330Ω, AlphaLib:0402R, symbol Device:R_Small
- removed R3: 8.2kΩ, AlphaLib:0402R, symbol Device:R_Small
- removed R3: 1.5kΩ, AlphaLib:0402R, symbol Device:R_Small
- removed SW9: SW_SPDT, corevus:MSS12C02-LS, symbol Switch:SW_SPDT
- removed U14: CD4504B, Package_SO:SOP-16_3.9x9.9mm_P1.27mm, symbol 4xxx:4504
- removed U15, U5: RT8110B, Package_TO_SOT_SMD:TSOT-23-8, symbol corevus:RT8110B
- removed U4: SRV05-4, Package_TO_SOT_SMD:SOT-23-6, symbol Power_Protection:SRV05-4
- removed U6: AMS1117-3.3, Package_TO_SOT_SMD:SOT-223-3_TabPin2, symbol Regulator_Linear:AMS1117-3.3
- added C10 (x11): 100nF 50V, AlphaLib:0402C, symbol Device:C_Small
- added C10: 120pF, AlphaLib:0402C, symbol Device:C_Small
- added C10 (x2): 100nF, AlphaLib:0402C, symbol Device:C_Small
- added C10 (x2): 10μF, AlphaLib:0603C, symbol Device:C_Small
- added C10: 12nF, AlphaLib:0402C, symbol Device:C_Small
- added C10: 2.2nF, AlphaLib:0402C, symbol Device:C_Small
- added C10: 36pF, AlphaLib:0402C, symbol Device:C_Small
- added C106, C108: 220μF 35V, Capacitor_THT:CP_Radial_D8.0mm_P3.50mm, symbol Device:C_Polarized_Small_US
- added C13 (x2): 22μF 25V, Capacitor_SMD:C_1206_3216Metric, symbol Device:C_Small
- added C13 (x2): 1μF, AlphaLib:0402C, symbol Device:C_Small
- added C13 (x2): 10μF 50V, Capacitor_SMD:C_1206_3216Metric, symbol Device:C_Small
- added D1 (x18): Red, AlphaLib:0402LED, symbol Device:LED_Small
- added D14, D29: 5819, Diode_SMD:D_SOD-123, symbol Device:D_Schottky_Small
- added D28: 1N5819, Diode_SMD:D_SOD-323, symbol Device:D_Schottky_Small
- added J15, J16, J2, J21, J22, J23, J4, J5: JST XH, corevus:JST_XH_1x02, symbol Connector:Conn_01x02_Pin
- added J18, J19, J20: 1x6P, corevus:PinHeader_1x06_P2.54mm_Vertical, symbol Connector:Conn_01x06_Pin
- added J24, J25, J26: XH, corevus:JST_XH_1x03, symbol Connector:Conn_01x03_Pin
- added J27: JST XH, corevus:JST_XH_1x03, symbol Connector:Conn_01x03_Pin
- added J29: USB_A, corevus:Jing_USB-A_906-761, symbol Connector:USB_A
- added J31 (x3): 1x2P, corevus:Kefa_KF8500-8.5-2P, symbol Connector:Screw_Terminal_01x02
- added J6: KK2.54, Connector:FanPinHeader_1x04_P2.54mm_Vertical, symbol Connector:Conn_01x04_Pin
- added L3: 22μH, corevus:L_Changjiang_FXL0640, symbol Device:L
- added Q1, Q19, Q2, Q20, Q21, Q23, Q24: AO3400, Package_TO_SOT_SMD:SOT-23, symbol Device:Q_NMOS_GSD
- added Q25, Q26: 60N03F, corevus:MOSFET_DFN8_5x6, symbol corevus:NMOS_DFN8
- added R3 (x19): 10kΩ, AlphaLib:0402R, symbol Device:R_Small
- added R3 (x12): 100Ω, AlphaLib:0402R, symbol Device:R_Small
- added R3: 270kΩ, AlphaLib:0402R, symbol Device:R_Small
- added R3: 23.7kΩ, AlphaLib:0402R, symbol Device:R_Small
- added R3 (x19): 4.7kΩ, AlphaLib:0402R, symbol Device:R_Small
- added R3: 47kΩ, AlphaLib:0402R, symbol Device:R_Small
- added R3: 100kΩ, AlphaLib:0402R, symbol Device:R_Small
- added R3: 3.74kΩ, AlphaLib:0402R, symbol Device:R_Small
- added R3 (x2): 22kΩ, AlphaLib:0402R, symbol Device:R_Small
- added R3: 5.6kΩ, AlphaLib:0402R, symbol Device:R_Small
- added R3 (x2): 250kΩ, AlphaLib:0402R, symbol Device:R_Small
- added R3: 30kΩ, AlphaLib:0402R, symbol Device:R_Small
- added R3: 3.3kΩ, AlphaLib:0402R, symbol Device:R_Small
- added SW4: SW_SPDT, corevus:MSS12C02-LS, symbol Switch:SW_SPDT
- added TH1, TH2, TH3: 10kΩ/3950K, AlphaLib:0402R, symbol Device:Thermistor_NTC
- added U2: CD4504B, Package_SO:SOP-16_3.9x9.9mm_P1.27mm, symbol 4xxx:4504
- added U3, U4: TPS54335A, Package_SO:SOIC-8-1EP_3.9x4.9mm_P1.27mm_EP2.95x4.9mm_Mask2.71x3.4mm_ThermalVias, symbol openbus:TPS54335A
- added U5: AMS1117-3.3, Package_TO_SOT_SMD:SOT-223-3_TabPin2, symbol Regulator_Linear:AMS1117-3.3
- H1, H2, H3, H4: footprint MountingHole:MountingHole_3.2mm_M3_Pad_Via -> MountingHole:MountingHole_3.2mm_M3_DIN965
- J14: value JST XH -> KK2.54; footprint corevus:JST_XH_1x04 -> Connector:FanPinHeader_1x04_P2.54mm_Vertical
- L1, L2: value 10μH -> 22μH; footprint corevus:CJiang_FXL1040 -> corevus:L_Changjiang_FXL0640
Connections:
- net +12V: now also SW2.1 (A), C108.1, C13.1, J20.1 (Pin_1), J20.2 (Pin_2), J20.3 (Pin_3), J20.4 (Pin_4), J20.5 (Pin_5), J20.6 (Pin_6), L3.2, R3.2; no longer L1.2
- net +24V: now also C13.1, C13.1, J18.1 (Pin_1), J18.2 (Pin_2), J18.3 (Pin_3), J18.4 (Pin_4), J18.5 (Pin_5), J18.6 (Pin_6), R3.1, R3.1, SW4.1 (A), U3.2 (VIN), U4.2 (VIN); no longer SW2.1 (A)
- net +3.3V: now also C10.1, C13.2, D1.2 (A), J24.3 (Pin_3), J25.3 (Pin_3), J26.3 (Pin_3), R3.2, R3.2, R3.2, R3.2, R3.2, R3.2, R3.2, U2.1 (VCC), U5.2 (VO)
- net +5V: now also C106.1, C13.1, D29.2 (A), J29.1 (VBUS), R3.2, SW4.3 (C); no longer SW2.3 (C)
- net Bed_H+: now also D14.1 (K), J31.1 (Pin_1)
- net Bed_H-: now also D14.2 (A), J31.2 (Pin_2), Q25.5 (D), Q25.6 (D), Q25.7 (D), Q25.8 (D), Q26.5 (D), Q26.6 (D), Q26.7 (D), Q26.8 (D)
- net F0: now also R3.1; no longer J14.4 (Pin_4), U1.56 (PG0)
- net F0_FG: now also J6.3 (Pin_3); no longer J14.3 (Pin_3), U1.57 (PG1)
- net F0_V+: now also C10.2, J19.1 (Pin_1), J6.2 (Pin_2); no longer J14.2 (Pin_2)
- net F1: now also R3.1; no longer U1.58 (PE7)
- net F1_FG: now also J14.3 (Pin_3); no longer U1.59 (PE8)
- net F1_V+: now also J14.2 (Pin_2), C10.2, J19.2 (Pin_2)
- net F2_Gate: now also R3.1; no longer Q22.1 (G), U1.60 (PE9)
- net F2_V+: now also C10.2, J19.3 (Pin_3), J2.2 (Pin_2); no longer J17.2 (Pin_2)
- net F3_Gate: now also R3.1; no longer U1.63 (PE10)
- net F3_V+: now also C10.2, J19.4 (Pin_4), J4.2 (Pin_2)
- net F4_Gate: now also R3.1; no longer Q28.1 (G), U1.64 (PE11)
- net F4_V+: now also C10.2, J19.5 (Pin_5), J5.2 (Pin_2)
- net F5_Gate: now also R3.1; no longer Q29.1 (G), U1.65 (PE12)
- net F5_V+: now also C10.2, J15.2 (Pin_2), J19.6 (Pin_6)
- net F6_Gate: now also R3.1; no longer Q30.1 (G), U1.66 (PE13)
- net F7_Gate: now also R3.1; no longer U1.67 (PE14)
- net F8_Gate: now also R3.1; no longer U1.68 (PE15)
- net GND: now also SW2.3 (C), C10.1, C10.1, C10.2, C10.2, C10.2, C10.2, C10.2, C10.2, C106.2, C108.2, C13.1, C13.1, C13.2, C13.2, C13.2, C13.2, J24.2 (Pin_2), J25.2 (Pin_2), J26.2 (Pin_2), J27.2 (Pin_2), J29.4 (GND), J31.1 (Pin_1), J31.1 (Pin_1), J6.1 (Pin_1), Q1.2 (S), Q19.2 (S), Q2.2 (S), Q20.2 (S), Q21.2 (S), Q23.2 (S), Q24.2 (S), Q25.1 (S), Q25.2 (S), Q25.3 (S), Q26.1 (S), Q26.2 (S), Q26.3 (S), R3.1, R3.1, R3.1, R3.2, R3.2, R3.2, R3.2, R3.2, R3.2, R3.2, R3.2, R3.2, R3.2, R3.2, R3.2, R3.2, R3.2, R3.2, R3.2, R3.2, R3.2, R3.2, R3.2, R3.2, R3.2, R3.2, R3.2, R3.2, R3.2, R3.2, R3.2, R3.2, R3.2, R3.2, R3.2, R3.2, R3.2, TH1.2, TH2.2, TH3.2, U2.13 (Select), U2.8 (VSS), U3.4 (GND), U3.9 (GND), U4.4 (GND), U4.9 (GND), U5.1 (GND)
- net H0: now also R3.1, U2.9 (Din); no longer U1.49 (PF11)
- net H0_Gate: now also U2.10 (Dout)
- net H1: now also R3.1, U2.11 (Ein); no longer U1.55 (PF15)
- net H1_Gate: now also U2.12 (Eout)
- net H2: now also R3.1, U2.3 (Ain); no longer U1.54 (PF14)
- net H2_Gate: now also U2.2 (Aout)
- net H3: now also R3.1, U2.5 (Bin); no longer U1.53 (PF13)
- net H3_Gate: now also U2.4 (Bout)
- net HB: now also R3.1, U2.14 (Fin); no longer U1.50 (PF12)
- net HB_Gate: now also R3.1, U2.15 (Fout)
- net T4: no longer U1.34 (PA0)
- net T5: no longer U1.35 (PA1)
- net USART2_RX: no longer U1.37 (PA3)
- net _{M0}Dir: no longer U1.113 (PC12)
- net _{M0}Step: no longer U1.114 (PD0)
- net _{M1}Dir: no longer U1.117 (PD3)
- net _{M1}Step: no longer U1.118 (PD4)
- net _{M4}Dir: no longer U1.142 (PE1)
- net _{M4}Step: no longer U1.139 (PB8)
- net at F2.1, F3.1, F5.1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: now also J31.2 (Pin_2)
- net at F1.1, F4.1: now also J31.2 (Pin_2)
- net at Q30.3 (D): now also C10.1, J23.1 (Pin_1)
- net at L1.1: now also C10.2, U3.3 (PH)
- net at J17.1 (Pin_1): now also C10.1, Q24.3 (D); no longer Q22.3 (D)
- net at Q28.3 (D): now also C10.1, J21.1 (Pin_1)
- net at Q29.3 (D): now also C10.1, J22.1 (Pin_1)
- net at L2.1: now also C10.2, U4.3 (PH)
- net at SW2.2 (B): now also C13.2, D1.2 (A), U2.16 (VDD)
- net VBUSDET: now reaches U1.101 (PA9)
- net E0: no longer names the net of U1.40 (PA4)
- net E1: no longer names the net of U1.20 (PF8)
- net E2: no longer names the net of U1.21 (PF9)
- net E3: no longer names the net of U1.22 (PF10)
- net USART2_TX: no longer names the net of U1.36 (PA2)
- net _{M0}UART: no longer names the net of U1.115 (PD1)
- net _{M0}~{En}: no longer names the net of U1.112 (PC11)
- net _{M10}Dir: no longer names the net of U1.2 (PE3)
- net _{M10}Step: no longer names the net of U1.1 (PE2)
- net _{M10}~{CS}: no longer names the net of U1.4 (PE5)
- net _{M10}~{En}: no longer names the net of U1.3 (PE4)
- net _{M12}Dir: no longer names the net of U1.7 (PC13)
- net _{M12}Step: no longer names the net of U1.5 (PE6)
- net _{M12}~{CS}: no longer names the net of U1.9 (PC15)
- net _{M12}~{En}: no longer names the net of U1.8 (PC14)
- net _{M1}UART: no longer names the net of U1.119 (PD5)
- net _{M1}~{En}: no longer names the net of U1.116 (PD2)
- net _{M20}Dir: no longer names the net of U1.11 (PF1)
- net _{M20}Step: no longer names the net of U1.10 (PF0)
- net _{M20}~{CS}: no longer names the net of U1.13 (PF3)
- net _{M20}~{En}: no longer names the net of U1.12 (PF2)
- net _{M22}Dir: no longer names the net of U1.15 (PF5)
- net _{M22}Step: no longer names the net of U1.14 (PF4)
- net _{M22}~{CS}: no longer names the net of U1.19 (PF7)
- net _{M22}~{En}: no longer names the net of U1.18 (PF6)
- net _{M2}Dir: no longer names the net of U1.123 (PD7)
- net _{M2}Step: no longer names the net of U1.124 (PG9)
- net _{M2}UART: no longer names the net of U1.125 (PG10)
- net _{M2}~{En}: no longer names the net of U1.122 (PD6)
- net _{M3}Dir: no longer names the net of U1.127 (PG12)
- net _{M3}Step: no longer names the net of U1.128 (PG13)
- net _{M3}UART: no longer names the net of U1.129 (PG14)
- net _{M3}~{En}: no longer names the net of U1.126 (PG11)
- net _{M4}Diag1: no longer names the net of U1.140 (PB9)
- net _{M4}~{CS}: no longer names the net of U1.137 (PB7)
- net _{M4}~{En}: no longer names the net of U1.141 (PE0)
- net _{M5}Diag1: no longer names the net of U1.136 (PB6)
- net _{M5}Dir: no longer names the net of U1.134 (PB4)
- net _{M5}Step: no longer names the net of U1.133 (PB3)
- net _{M5}~{CS}: no longer names the net of U1.132 (PG15)
- net _{M5}~{En}: no longer names the net of U1.135 (PB5)
- new net: J14.4 (Pin_4), Q21.3 (D)
- new net: C10.1, J2.1 (Pin_1), Q1.3 (D)
- new net: D1.2 (A), Q20.1 (G), R3.1, R3.2
- new net: C10.1, R3.2, U4.6 (COMP)
- new net: C10.1, U3.1 (BOOT)
- new net: D1.2 (A), Q19.1 (G), R3.1, R3.2
- new net: R3.1, R3.2, U3.7 (EN)
- new net: D1.2 (A), Q1.1 (G), R3.1, R3.2
- new net: C10.1, R3.1 (x2)
- new net: C10.1, R3.2, U3.6 (COMP)
- new net: D1.2 (A), Q2.1 (G), R3.1, R3.2
- new net: C10.1, J4.1 (Pin_1), Q2.3 (D)
- new net: D1.1 (K), R3.2 (x3)
- new net: D1.2 (A), R3.1 (x4)
- new net: D1.2 (A), Q28.1 (G), R3.1, R3.2
- new net: D1.2 (A), Q30.1 (G), R3.1, R3.2
- new net: D1.2 (A), Q29.1 (G), R3.1, R3.2
- new net: C10.1, U4.1 (BOOT)
- new net: R3.1, R3.1, U4.5 (VSENSE)
- new net: R3.1, R3.2, U4.7 (EN)
- new net: R3.1, U4.8 (RT)
- new net: D1.1 (K), R3.1 (x11)
- new net: R3.1, R3.1, U3.5 (VSENSE)
- new net: C10.1, J16.1 (Pin_1), Q23.3 (D)
- new net: D1.2 (A), Q24.1 (G), R3.1, R3.2
- new net: D1.2 (A), Q25.4 (G), Q26.4 (G), R3.2
- new net: D1.2 (A), Q22.1 (G), R3.1, R3.2
- new net: D1.2 (A), Q23.1 (G), R3.1, R3.2
- new net: D28.1 (K), J27.1 (Pin_1)
- new net: J27.3 (Pin_3), SW4.2 (B)
- new net: J6.4 (Pin_4), Q20.3 (D)
- new net: D1.2 (A), Q21.1 (G), R3.1, R3.2
- new net: L1.2, L3.1
- new net: C10.1, J15.1 (Pin_1), Q22.3 (D)
- new net: R3.1, U3.8 (RT)
- new net: C10.1, J5.1 (Pin_1), Q19.3 (D)
- new net F10_Gate: R3.1
- new net F10_V+: C10.2, J23.2 (Pin_2)
- new net F6_V+: C10.2, J16.2 (Pin_2)
- new net F7_V+: C10.2, J17.2 (Pin_2)
- new net F8_V+: C10.2, J21.2 (Pin_2)
- new net F9_Gate: R3.1
- new net F9_V+: C10.2, J22.2 (Pin_2)
- new net H4: R3.1, U2.7 (Cin)
- new net H4_Gate: U2.6 (Cout)
- new net S0: D1.1 (K), J24.1 (Pin_1)
- new net S1: D1.1 (K), J25.1 (Pin_1)
- new net S2: D1.1 (K), J26.1 (Pin_1)
- new net S3: D1.1 (K), D28.2 (A)
- new net USB_VBUS: C10.1, D29.1 (K), U5.3 (VI)
- new net _{M1}~{Therm}: R3.1, TH2.1
- new net _{M4}~{Therm}: R3.1, TH3.1
- new net _{PWR}~{Therm}: R3.1, TH1.1
- no-connect marks 8 -> 9
Other:
- sheet Motor 0 (TMC2208) renamed Motor 4 (TMC2208)
- sheet Motor 1 (TMC2208) renamed Motor 5 (TMC2208)
- sheet Motor 2 (TMC2208) renamed Motor 6 (TMC2208)
- sheet Motor 3 (TMC2208) renamed Motor 7 (TMC2208)
- sheet Motor 4 (TMCx160) renamed Motor 0 (TMC2160)
- sheet Motor 5 (TMCx160) renamed Motor 1 (TMC2160)
- sheet Motor Expansion 1x renamed Motor Expansion 2A, 2B
- sheet Motor Expansion 2x renamed Motor Expansion 3A, 3B
- removed sheet Pi Zero + USB Hub
- added sheet Heater 4 (driver_heater.kicad_sch)
- sheet Motor 0 (TMC2160): file driver-tmc5160-integrated.kicad_sch -> driver-tmc2160-integrated.kicad_sch
- sheet Motor 0 (TMC2160) ports: added none; removed Clk, ENCA, ENCB, ENCN
- sheet Motor 1 (TMC2160): file driver-tmc5160-integrated.kicad_sch -> driver-tmc2160-integrated.kicad_sch
- sheet Motor 1 (TMC2160) ports: added none; removed Clk, ENCA, ENCB, ENCN
- sheet Motor Expansion 2A, 2B ports: added Therm, _{MA}Diag, _{MA}Dir, _{MA}Step, _{MA}~{CS}, _{MA}~{En}, _{MB}Diag, _{MB}Dir, _{MB}Step, _{MB}~{CS}, _{MB}~{En}; removed Clk, _{M0}Diag0, _{M0}Diag1, _{M0}Dir, _{M0}Step, _{M0}~{CS}, _{M0}~{En}, _{M2}Diag0, _{M2}Diag1, _{M2}Dir, _{M2}Step, _{M2}~{CS}, _{M2}~{En}
- sheet Motor Expansion 3A, 3B ports: added Therm, _{MA}Diag, _{MA}Dir, _{MA}Step, _{MA}~{CS}, _{MA}~{En}, _{MB}Diag, _{MB}Dir, _{MB}Step, _{MB}~{CS}, _{MB}~{En}; removed Clk, _{M0}Diag0, _{M0}Diag1, _{M0}Dir, _{M0}Step, _{M0}~{CS}, _{M0}~{En}, _{M2}Diag0, _{M2}Diag1, _{M2}Dir, _{M2}Step, _{M2}~{CS}, _{M2}~{En}
- note removed: "12.2V"
- note removed: "5.16V"
- note removed: "Endstops"
- note removed: "four low-power stepper channels, two high-power (TMCx160) stepper channels supporting max. 60V 5A, and and two discrete-element LGA sockets provisioned to accommodate up to four drivers per socket, for up to a maximum of fourteen stepper channels."
- moved on the sheet: C10, C12, C13, C14, C16, C17, D1, F1, F2, F3, F4, F5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

Commit message: v0.4 mostly complete, board needs minor revisions (e.g. pin swap)
Parts:
- removed C10 (x3): 100nF 50V, AlphaLib:0402C, symbol Device:C_Small
- removed D1 (x3): Red, AlphaLib:0402LED, symbol Device:LED_Small
- removed J13: EXP1, Connector_IDC:IDC-Header_2x05_P2.54mm_Vertical, symbol Connector_Generic:Conn_02x05_Odd_Even
- removed J18, J19, J20: 1x6P, corevus:PinHeader_1x06_P2.54mm_Vertical, symbol Connector:Conn_01x06_Pin
- removed J28: EXP2, Connector_IDC:IDC-Header_2x05_P2.54mm_Vertical, symbol Connector_Generic:Conn_02x05_Odd_Even
- removed L3: 22μH, corevus:L_Changjiang_FXL0640, symbol Device:L
- removed NT2: NetTie_2, corevus:NetTie-2_SMD_Pad0.1mm, symbol Device:NetTie_2
- removed Q30: AO3400, Package_TO_SOT_SMD:SOT-23, symbol Device:Q_NMOS_GSD
- removed R3 (x3): 10kΩ, AlphaLib:0402R, symbol Device:R_Small
- removed R3: 100Ω, AlphaLib:0402R, symbol Device:R_Small
- removed R3: 1kΩ, AlphaLib:0402R, symbol Device:R_Small
- removed R3: 4.7kΩ, AlphaLib:0402R, symbol Device:R_Small
- removed SW1, SW2, SW4: SW_SPDT, corevus:MSS12C02-LS, symbol Switch:SW_SPDT
- added C109: 220μF 35V, Capacitor_THT:CP_Radial_D8.0mm_P3.50mm, symbol Device:C_Polarized_Small_US
- added C68, C69, C70, C71, C72, C73: 1μF, AlphaLib:0402C, symbol Device:C_Small
- added J13: USB 2.0, corevus:USB_Type-C_16p, symbol Connector:USB_C_Receptacle_USB2.0
- added J18, J19, J20, J31, J38: 1x3P, corevus:PinHeader_1x03_P2.54mm_Vertical, symbol Connector:Conn_01x03_Pin
- added J28: MF3, corevus:Molex_Micro-Fit-3.0_430450813, symbol Connector_Generic:Conn_02x04_Top_Bottom
- added J37: 2x05P, Connector_PinHeader_1.27mm:PinHeader_2x05_P1.27mm_Vertical, symbol Connector_Generic:Conn_02x05_Odd_Even
- added J39: JST XH, corevus:JST_XH_1x02, symbol Connector:Conn_01x02_Pin
- added R12, R2, R3: 4.7kΩ, AlphaLib:0402R, symbol Device:R_Small
- added R3 (x2): 5.1kΩ, AlphaLib:0402R, symbol Device:R_Small
- added SW1: SPST, corevus:XKB_TS-1187A, symbol Switch:SW_Push
- added TH4: 10kΩ/3950K, AlphaLib:0402R, symbol Device:Thermistor_NTC
- C10: value 100nF -> 1µF
- C10: value 10μF -> 1μF; footprint AlphaLib:0603C -> AlphaLib:0402C; LCSC C19702 -> (none)
- C12: value 470μF 63V -> 220μF 35V; footprint corevus:CP_Radial_D12.5mm_P5.00mm -> Capacitor_THT:CP_Radial_D8.0mm_P3.50mm; Field4 C310848 -> (none)
- L1: value 22μH -> 47μH; footprint corevus:L_Changjiang_FXL0640 -> corevus:L_Changjiang_FXL1040
- R3: footprint AlphaLib:0402R -> AlphaLib:0603R
- renumbered H5 to H13, J31 to J3, J31 to J35, J31 to J36
Connections:
- net Btn_En1 is gone; now on net _{M0}CS: U1.91 (PG6)
- net Btn_En2 is gone; now on net _{M0}Dir: U1.92 (PG7)
- net Btn_Enc is gone; now on net _{M0}Diag1: U1.89 (PG4)
- net Buzzer is gone; now on net _{M0}En: U1.90 (PG5)
- net F0_V+ is gone; now on net +12V: J6.2 (Pin_2)
- net F10_V+ is gone; now on net T6: J23.2 (Pin_2)
- net F1_V+ is gone; now on net +12V: J14.2 (Pin_2)
- net F6_V+ is gone; now on net +12V: C10.2, J16.2 (Pin_2)
- net F7_V+ is gone; now on net +12V: C10.2, J17.2 (Pin_2)
- net F8_V+ is gone; now on net +12V: C10.2, J21.2 (Pin_2)
- net F9_V+ is gone; now on net +5V: C10.2, J22.2 (Pin_2)
- net H4 is gone; now on net GND: U2.7 (Cin)
- net LCD_D4 is gone; now on net _{M1}Step: U1.86 (PD15)
- net LCD_D5 is gone; now on net _{M1}En: U1.85 (PD14)
- net LCD_D6 is gone; now on net _{M1}Diag1: U1.82 (PD13)
- net LCD_D7 is gone; now on net _{M2B}Step: U1.81 (PD12)
- net LCD_En is gone; now on net _{M1}CS: U1.88 (PG3)
- net LCD_Rs is gone; now on net _{M2B}Dir: U1.80 (PD11)
- net SD_CS is gone; now on net _{M0}Step: U1.93 (PG8)
- net SD_Det is gone; now on net _{M1}Dir: U1.87 (PG2)
- net VBUSDET is gone; now on net +3.3V: U1.101 (PA9)
- net _{M1}~{Therm} is gone; now on net _{M1}Therm: R3.1, TH2.1
- net _{M4}~{Therm} is gone; now on net _{M4}Therm: R3.1, TH3.1
- net _{PWR}~{Therm} is gone; now on net _{12V}Therm: R3.1, TH1.1
- net +12V: now also C13.2, L1.2, U2.16 (VDD), J18.1 (Pin_1), J19.1 (Pin_1), J20.1 (Pin_1), J28.7 (Pin_7), J31.1 (Pin_1)
- net +24V: now also C109.1, J18.3 (Pin_3), J19.3 (Pin_3), J20.3 (Pin_3), J28.5 (Pin_5), J28.6 (Pin_6), J31.3 (Pin_3), J38.1 (Pin_1)
- net +3.3V: now also J37.1 (Pin_1), R3.2, SW1.2; no longer C10.1, J24.3 (Pin_3), J25.3 (Pin_3), J26.3 (Pin_3), R3.2, R3.2, R3.2, R3.2
- net +5V: now also J24.3 (Pin_3), J25.3 (Pin_3), J26.3 (Pin_3), R3.2, R3.2, R3.2, R3.2, J38.3 (Pin_3)
- net BOOT0: now also SW1.1
- net F0: now also U1.102 (PA10)
- net F0_FG: now also U1.112 (PC11)
- net F1: now also U1.110 (PA15)
- net F1_FG: now also U1.111 (PC10)
- net F2_Gate: now also U1.134 (PB4)
- net F2_V+: now also J18.2 (Pin_2)
- net F3_Gate: now also U1.133 (PB3)
- net F3_V+: now also J20.2 (Pin_2)
- net F4_Gate: now also U1.136 (PB6)
- net F4_V+: now also J19.2 (Pin_2)
- net F5_Gate: now also U1.135 (PB5)
- net F5_V+: now also J31.2 (Pin_2)
- net F6_Gate: now also U1.140 (PB9)
- net F7_Gate: now also U1.139 (PB8)
- net F8_Gate: now also U1.5 (PE6)
- net F9_Gate: now also U1.137 (PB7)
- net GND: now also C109.2, C68.1, C69.1, C70.1, C71.1, J13.A1 (GND), J13.A12 (GND), J13.B1 (GND), J13.B12 (GND), J13.S1 (SHIELD), J28.1 (Pin_1), J28.2 (Pin_2), J28.3 (Pin_3), J37.3 (Pin_3), J37.5 (Pin_5), J37.9 (Pin_9), R3.2, R3.2, TH4.2; no longer C10.2
- net H0: now also R3.1, U1.115 (PD1), U2.11 (Ein); no longer R3.1, U2.9 (Din)
- net H0_Gate: now also U2.12 (Eout); no longer U2.10 (Dout)
- net H1: now also R3.1, U1.114 (PD0), U2.9 (Din); no longer R3.1, U2.11 (Ein)
- net H1_Gate: now also U2.10 (Dout); no longer U2.12 (Eout)
- net H2: now also U1.117 (PD3)
- net H3: now also U1.118 (PD4)
- net HB: now also U1.116 (PD2)
- net S0: now also U1.127 (PG12)
- net S1: now also U1.128 (PG13)
- net S2: now also U1.129 (PG14)
- net S3: now also U1.132 (PG15)
- net T0: now also C10.2, J11.2 (Pin_2), R3.1, U1.34 (PA0); no longer C10.2, J8.2 (Pin_2), R3.1, U1.26 (PC0)
- net T1: now also C10.2, J10.2 (Pin_2), R3.1, U1.35 (PA1); no longer C10.2, J7.2 (Pin_2), R3.1, U1.27 (PC1)
- net T3: now also C10.2, J12.2 (Pin_2), R3.1; no longer C10.2, J10.2 (Pin_2), R3.1
- net T4: now also C10.2, J8.2 (Pin_2), R3.1, U1.26 (PC0); no longer C10.2, J11.2 (Pin_2), R3.1
- net T5: now also C10.2, J7.2 (Pin_2), R3.1, U1.27 (PC1); no longer C10.2, J12.2 (Pin_2), R3.1
- net USART2_RX: now also U1.37 (PA3)
- net USB_VBUS: now also J1.A4 (VBUS), J1.A9 (VBUS), J1.B4 (VBUS), J1.B9 (VBUS)
- net VDDA: now also C10.1, U1.32 (VREF+), R12.2, R2.2
- net VSSA: now also C10.2, J23.1 (Pin_1), C72.1, C73.1, J39.1 (Pin_1)
- net _{M2A}CS: now also U1.67 (PE14)
- net _{M2A}Diag: now also U1.68 (PE15)
- net _{M2A}Dir: now also U1.65 (PE12)
- net _{M2A}En: now also U1.66 (PE13)
- net _{M2A}Step: now also U1.73 (PB12)
- net _{M2B}CS: now also U1.78 (PD9)
- net _{M2B}Diag: now also U1.77 (PD8)
- net _{M2B}En: now also U1.79 (PD10)
- net _{M2}Therm: now also U1.46 (PB0)
- net _{M3A}CS: now also U1.57 (PG1)
- net _{M3A}Diag: now also U1.56 (PG0)
- net _{M3A}Dir: now also U1.54 (PF14)
- net _{M3A}En: now also U1.55 (PF15)
- net _{M3A}Step: now also U1.53 (PF13)
- net _{M3B}CS: now also U1.59 (PE8)
- net _{M3B}Diag: now also U1.58 (PE7)
- net _{M3B}Dir: now also U1.63 (PE10)
- net _{M3B}En: now also U1.60 (PE9)
- net _{M3B}Step: now also U1.64 (PE11)
- net _{M4}Dir: now also U1.44 (PC4)
- net _{M4}En: now also U1.45 (PC5)
- net _{M4}Step: now also U1.49 (PF11)
- net _{M4}UART: now also U1.50 (PF12)
- net ~{Reset}: now also J37.10 (Pin_10)
- net at J27.3 (Pin_3): now also J38.2 (Pin_2)
- net USB_D+: now reaches R3.1, U1.104 (PA12)
- net USB_D-: now reaches R3.1, U1.103 (PA11)
- net _{M7}Dir: now reaches U1.1 (PE2)
- net _{M6}UART: now reaches U1.10 (PF0)
- net SWDIO: now reaches U1.105 (PA13)
- net SWDIO: now also J37.2 (Pin_2)
- net SWCLK: now reaches U1.109 (PA14)
- net SWCLK: now also J37.4 (Pin_4)
- net _{M5}Dir: now reaches U1.11 (PF1)
- net _{M5}En: now reaches U1.12 (PF2)
- net _{M5}Step: now reaches U1.13 (PF3)
- net _{M5}UART: now reaches U1.14 (PF4)
- net T6: now reaches U1.18 (PF6)
- net T6: now also C72.2, R2.1
- net T7: now reaches U1.19 (PF7)
- net T7: now also C73.2, J39.2 (Pin_2), R12.1
- net _{M7}En: now reaches U1.2 (PE3)
- net _{M3}Therm: now reaches U1.20 (PF8)
- net _{5V}Therm: now reaches U1.21 (PF9)
- net _{5V}Therm: now also C71.2, R3.1, TH4.1
- net _{12V}Therm: now reaches U1.22 (PF10)
- net _{12V}Therm: now also C68.2
- net _{M7}Step: now reaches U1.3 (PE4)
- net USART2_TX: now reaches U1.36 (PA2)
- net _{M7}UART: now reaches U1.4 (PE5)
- net _{M4}Therm: now reaches U1.40 (PA4)
- net _{M4}Therm: now also C70.2
- net _{M1}Therm: now reaches U1.47 (PB1)
- net _{M1}Therm: now also C69.2
- net _{M6}Dir: now reaches U1.7 (PC13)
- net _{M6}En: now reaches U1.8 (PC14)
- net _{M6}Step: now reaches U1.9 (PC15)
- net H4_Gate: no longer names the net of U2.6 (Cout)
- new net: J13.A5 (CC1), R3.1
- new net: J13.A4 (VBUS), J13.A9 (VBUS), J13.B4 (VBUS), J13.B9 (VBUS)
- new net: J13.B5 (CC2), R3.1
- new net TH_USB_D+: J13.A6 (D+), J13.B6 (D+), J28.8 (Pin_8)
- new net TH_USB_D-: J13.A7 (D-), J13.B7 (D-), J28.4 (Pin_4)
- no-connect marks 9 -> 15
Other:
- removed sheet Heater 4
- moved on the sheet: C10, C106, C108, C13, C14, C16, C17, D1, D29, FB1, H13, J10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

Commit message: CvG v0.4 complete, now updating documentation
Parts:
- added H? (x2): ToolingHole, corevus:ToolingHole, symbol Mechanical:MountingHole
- C10: value 120pF -> 100pF
- C10: value 12nF -> 10nF
- C10: value 36pF -> 33pF
- C106, C108: value 220μF 35V -> 220μF 25V
- R3: value 270kΩ -> 220kΩ
- R3: value 23.7kΩ -> 24kΩ
- R3: value 3.74kΩ -> 4.7kΩ
- R3: value 250kΩ -> 220kΩ
- R3: value 22kΩ -> 18kΩ
Other:
- moved on the sheet: J13, J28, R3

Commit message: non-working commit, moved around various connectors etc in preparation for v0.5
Parts:
- removed J37: 2x05P, Connector_PinHeader_1.27mm:PinHeader_2x05_P1.27mm_Vertical, symbol Connector_Generic:Conn_02x05_Odd_Even
- added C74, C75: 100nF 50V, AlphaLib:0402C, symbol Device:C_Small
- added D1, D7, D? (x2): Red, AlphaLib:0402LED, symbol Device:LED_Small
- added J37, J40: JST XH, corevus:JST_XH_1x02, symbol Connector:Conn_01x02_Pin
- added J41, J42: 1x3P, corevus:PinHeader_1x03_P2.54mm_Vertical, symbol Connector:Conn_01x03_Pin
- added Q27, Q30: AO3400, Package_TO_SOT_SMD:SOT-23, symbol Device:Q_NMOS_GSD
- added R126, R127, R? (x2): 4.7kΩ, AlphaLib:0402R, symbol Device:R_Small
- added R59, R76: 100Ω, AlphaLib:0402R, symbol Device:R_Small
- added R79, R82: 10kΩ, AlphaLib:0402R, symbol Device:R_Small
- J28: value MF3 -> MF3 2x04P
- gave numbers to parts that had none: 2
Connections:
- net +12V: now also J28.6 (Pin_6), J41.1 (Pin_1), J42.1 (Pin_1), R?.2; no longer C10.2, J21.2 (Pin_2), J28.7 (Pin_7)
- net +24V: now also J28.7 (Pin_7), J28.8 (Pin_8), J41.3 (Pin_3), J42.3 (Pin_3); no longer J28.5 (Pin_5), J28.6 (Pin_6)
- net +5V: now also C10.2, J21.2 (Pin_2), R?.2
- net F4_Gate: now also R59.1; no longer R3.1
- net F4_V+: now also C74.2, J37.2 (Pin_2); no longer C10.2, J5.2 (Pin_2)
- net F5_Gate: now also R3.1; no longer R3.1
- net F5_V+: now also C10.2, J5.2 (Pin_2); no longer C10.2, J15.2 (Pin_2)
- net F6_Gate: now also R3.1; no longer R3.1
- net F7_Gate: now also R76.1; no longer R3.1
- net F8_Gate: now also R3.1; no longer R3.1
- net F9_Gate: now also R3.1; no longer R3.1
- net GND: now also J28.4 (Pin_4), D?.1 (K), D?.1 (K), Q27.2 (S), Q30.2 (S), R126.2, R127.2, R79.2, R82.2; no longer J28.1 (Pin_1)
- net H0: now also U1.97 (PC7); no longer U1.115 (PD1)
- net H1: now also U1.96 (PC6); no longer U1.114 (PD0)
- net H2: now also U1.99 (PC9); no longer U1.117 (PD3)
- net H3: now also U1.100 (PA8); no longer U1.118 (PD4)
- net HB: now also U1.98 (PC8); no longer U1.116 (PD2)
- net S0: now also U1.129 (PG14); no longer U1.127 (PG12)
- net S1: now also U1.132 (PG15); no longer U1.128 (PG13)
- net S2: now also U1.141 (PE0); no longer U1.129 (PG14)
- net S3: now also U1.142 (PE1); no longer U1.132 (PG15)
- net T0: now also U1.22 (PF10); no longer U1.34 (PA0)
- net T6: now also U1.15 (PF5); no longer U1.18 (PF6)
- net T7: now also U1.18 (PF6); no longer U1.19 (PF7)
- net TH_USB_D+: now also J28.5 (Pin_5); no longer J28.8 (Pin_8)
- net TH_USB_D-: now also J28.1 (Pin_1); no longer J28.4 (Pin_4)
- net _{12V}Therm: now also U1.20 (PF8); no longer U1.22 (PF10)
- net _{5V}Therm: now also U1.19 (PF7); no longer U1.21 (PF9)
- net _{M3}Therm: now also U1.21 (PF9); no longer U1.20 (PF8)
- new net: D?.2 (A), R?.1 (x2)
- new net: C75.1, J40.1 (Pin_1), Q30.3 (D)
- new net: D1.2 (A), Q27.1 (G), R59.2, R79.1
- new net: C74.1, J37.1 (Pin_1), Q27.3 (D)
- new net: D7.1 (K), R127.1
- new net: D7.2 (A), Q30.1 (G), R76.2, R82.1
- new net: D1.1 (K), R126.1
- new net DFU_ON: U1.114 (PD0)
- new net F10_Gate: R3.1
- new net F11_Gate: R3.1
- new net F6_V+: C10.2, J15.2 (Pin_2), J41.2 (Pin_2)
- new net F7_V+: C75.2, J40.2 (Pin_2), J42.2 (Pin_2)
- no-connect marks 15 -> 12
Other:
- moved on the sheet: C10, D1, D28, J16, J17, J21, J22, J24, J25, J26, J27, J28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

Commit message: corevus toolboard v0.2 release (working), corevus-g v0.2 release (very much not working), m++ v0.1 (not working, needs a lot of bodges)
Parts:
- removed C10: 1µF, AlphaLib:0402C, symbol Device:C_Small
- removed C10: 100pF, AlphaLib:0402C, symbol Device:C_Small
- removed C10: 100nF, AlphaLib:0402C, symbol Device:C_Small
- removed C10: 10nF, AlphaLib:0402C, symbol Device:C_Small
- removed C10: 2.2nF, AlphaLib:0402C, symbol Device:C_Small
- removed C10: 33pF, AlphaLib:0402C, symbol Device:C_Small
- removed C13: 10μF 50V, Capacitor_SMD:C_1206_3216Metric, symbol Device:C_Small
- removed R3 (x3): 220kΩ, AlphaLib:0402R, symbol Device:R_Small
- removed R3: 24kΩ, AlphaLib:0402R, symbol Device:R_Small
- removed R3: 100kΩ, AlphaLib:0402R, symbol Device:R_Small
- removed R3: 4.7kΩ, AlphaLib:0402R, symbol Device:R_Small
- removed R3: 22kΩ, AlphaLib:0402R, symbol Device:R_Small
- removed R3: 18kΩ, AlphaLib:0402R, symbol Device:R_Small
- removed U3, U4: TPS54335A, Package_SO:SOIC-8-1EP_3.9x4.9mm_P1.27mm_EP2.95x4.9mm_Mask2.71x3.4mm_ThermalVias, symbol openbus:TPS54335A
- added C100, C88: 100nF, AlphaLib:0402C, symbol Device:C_Small
- added C80, C98: 1µF, AlphaLib:0402C, symbol Device:C_Small
- added C86, C95: 22μF 25V, Capacitor_SMD:C_1206_3216Metric, symbol Device:C_Small
- added C94: 10μF 50V, Capacitor_SMD:C_1206_3216Metric, symbol Device:C_Small
- added D37: Grn, AlphaLib:0402LED, symbol Device:LED_Small
- added NT2, NT7: NetTie_2, corevus:NetTie-2_SMD_Pad0.1mm, symbol Device:NetTie_2
- added R130: 4.7kΩ, AlphaLib:0402R, symbol Device:R_Small
- added R90: 15kΩ, AlphaLib:0402R, symbol Device:R_Small
- added R92, R93: 330kΩ, AlphaLib:0402R, symbol Device:R_Small
- added U3, U4: AOZ1267QI-01, corevus:AOZ1267QI, symbol corevus:AOZ1267QI-01
- C10: value 15pF -> 16pF
- D1: value Red -> Grn
- D17, D32: renamed from D?; value Red -> Grn
- D28: footprint Diode_SMD:D_SOD-323 -> corevus:D_SOD-323
- L1: value 47μH -> 6.8μH
- L2: value 22μH -> 4.7μH
- R3: footprint AlphaLib:0603R -> AlphaLib:0402R
- R3: value 100kΩ -> 1kΩ
- R3: value 30kΩ -> 15kΩ; footprint AlphaLib:0603R -> AlphaLib:0402R
- SW1, SW3: footprint corevus:XKB_TS-1187A -> corevus:BZCN_TSC015
- Y1: value 12 MHz -> 25 MHz
- gave numbers to parts that had none: 2
Connections:
- net +12V: now also C95.1
- net +24V: now also C94.1, R92.1, R93.1, U3.22 (In), U3.7 (AIn), U3.8 (In), U3.9 (In), U4.22 (In), U4.7 (AIn), U4.8 (In), U4.9 (In)
- net +3.3V: now also R3.2; no longer D1.2 (A)
- net +5V: now also C86.1, R90.2; no longer R3.2
- net DFU_ON: now also R130.2
- net F0: now also U1.134 (PB4); no longer U1.102 (PA10)
- net F1: now also U1.133 (PB3); no longer U1.110 (PA15)
- net F10_Gate: now also U1.5 (PE6)
- net F11_Gate: now also U1.137 (PB7)
- net F2_Gate: now also U1.135 (PB5); no longer U1.134 (PB4)
- net F3_Gate: now also U1.127 (PG12); no longer U1.133 (PB3)
- net F4_Gate: now also U1.102 (PA10); no longer U1.136 (PB6)
- net F5_Gate: now also U1.136 (PB6); no longer U1.135 (PB5)
- net F6_Gate: now also U1.128 (PG13); no longer U1.140 (PB9)
- net F7_Gate: now also U1.110 (PA15); no longer U1.139 (PB8)
- net F8_Gate: now also U1.140 (PB9); no longer U1.5 (PE6)
- net F9_Gate: now also U1.139 (PB8); no longer U1.137 (PB7)
- net GND: now also D1.1 (K), D1.1 (K), D1.1 (K), C100.1, C80.1, C86.2, C88.1, C94.2, C95.2, C98.1, D37.1 (K), NT2.1, NT7.1, U3.12 (PGnd), U3.13 (PGnd), U3.14 (PGnd), U3.15 (PGnd), U3.19 (PGnd), U3.3 (~{PFM}), U4.12 (PGnd), U4.13 (PGnd), U4.14 (PGnd), U4.15 (PGnd), U4.19 (PGnd), U4.3 (~{PFM}); no longer R3.1, R3.2, R3.2, R3.2, R3.2
- net S0: now also U1.125 (PG10); no longer U1.129 (PG14)
- net at Q20.1 (G), R3.1, R3.2: now also R3.2; no longer D1.2 (A)
- net at C10.1: now also U3.20 (Bst)
- net at C10.2, L1.1: now also U3.10 (Lx), U3.11 (Lx), U3.16 (Lx), U3.17 (Lx), U3.18 (Lx)
- net at C10.1: now also U4.20 (Bst)
- net at C10.2, L2.1: now also U4.10 (Lx), U4.11 (Lx), U4.16 (Lx), U4.17 (Lx), U4.18 (Lx)
- net at R3.1, R3.1: now also U4.5 (FB)
- net at C10.2, Y1.3: now also R3.1; no longer R3.2, U1.24 (PH1)
- net at R3.1, R3.1: now also U3.5 (FB)
- net at R3.1: now also Q21.1 (G), R3.1, R3.2; no longer D1.1 (K)
- net at C10.2, U1.23 (PH0), Y1.1: no longer R3.1
- net at R3.1: now also D1.2 (A); no longer D1.1 (K)
- new net: D37.2 (A), R130.1
- new net: D1.2 (A), R3.1
- new net: D1.2 (A), R3.2
- new net: NT2.2, R3.2, U4.4 (AGnd)
- new net: R92.2, U4.6 (TOn)
- new net: C88.2, U4.23 (SS)
- new net: R3.2, U1.24 (PH1)
- new net: NT7.2, R3.2, U3.4 (AGnd)
- new net: R3.2, R90.1
- new net: C100.2, U3.23 (SS)
- new net: C98.2, U3.2 (En), U3.21 (V_{CC})
- new net: R93.2, U3.6 (TOn)
- new net: C80.2, U4.2 (En), U4.21 (V_{CC})
- no-connect marks 12 -> 22
Other:
- sheet Motor 4 (TMC2208) renamed Motor 4 (TMC2209)
- removed sheet Motor 5 (TMC2208)
- removed sheet Motor 6 (TMC2208)
- removed sheet Motor 7 (TMC2208)
- added sheet Motor 5 (TMC2209) (driver-tmc2209-integrated.kicad_sch)
- added sheet Motor 6 (TMC2209) (driver-tmc2209-integrated.kicad_sch)
- added sheet Motor 7 (TMC2209) (driver-tmc2209-integrated.kicad_sch)
- sheet Motor 4 (TMC2209): file driver-tmc2208-integrated.kicad_sch -> driver-tmc2209-integrated.kicad_sch
- note added: "EXPERIMENTAl"
- note added: "Todo: consider 9.5mm pitch 1x6"
- note removed: "0.8V"
- note removed: "Capacitor dissipation resistors"
- moved on the sheet: C10, C106, C108, C13, C68, C69, C70, C71, C72, C73, C74, C75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
