File: hardware/corevus-g/corevus-g.kicad_sch (KiCad schematic)
At the start: 256 parts, among them J1 USB 2.0, J10 JST XH, J11 JST XH, J12 JST XH, J13 USB 2.0, J14 KK2.54, J15 JST XH, J16 JST XH, J17 JST XH, J18 1x3P, J19 1x3P, J2 JST XH, J20 1x3P, J21 JST XH, J22 JST XH, J23 JST XH, J24 XH, J25 XH, J26 XH, J27 JST XH, J28 MF3 2x04P, J29 USB_A, J3 1x2P, J31 1x3P, J35 1x2P, J36 1x2P, J37 JST XH, J38 1x3P, J39 JST XH, J4 JST XH, J40 JST XH, J41 1x3P, J42 1x3P, J5 JST XH, J6 KK2.54, J7 JST XH, J8 JST XH, J9 JST XH, Q1 AO3400, Q19 AO3400, Q2 AO3400, Q20 AO3400, Q21 AO3400, Q22 AO3400, Q23 AO3400, Q24 AO3400, Q25 60N03F, Q26 60N03F, Q27 AO3400, Q28 AO3400, Q29 AO3400, Q30 AO3400, SW1 SPST, SW3 SPST, U1 STM32F407ZETx, U2 CD4504B, U3 AOZ1267QI-01, U4 AOZ1267QI-01, U5 AMS1117-3.3, Y1 25 MHz

Commit message: why not
Parts:
- removed C10 (x2), C100: 100nF, AlphaLib:0402C, symbol Device:C_Small
- removed C13: 1μF, AlphaLib:0402C, symbol Device:C_Small
- removed D37: Grn, AlphaLib:0402LED, symbol Device:LED_Small
- removed NT2, NT7: NetTie_2, corevus:NetTie-2_SMD_Pad0.1mm, symbol Device:NetTie_2
- removed R130: 4.7kΩ, AlphaLib:0402R, symbol Device:R_Small
- removed R3: 47kΩ, AlphaLib:0402R, symbol Device:R_Small
- removed R3: 5.6kΩ, AlphaLib:0402R, symbol Device:R_Small
- removed R3: 15kΩ, AlphaLib:0402R, symbol Device:R_Small
- removed R3: 3.3kΩ, AlphaLib:0402R, symbol Device:R_Small
- removed U3, U4: AOZ1267QI-01, corevus:AOZ1267QI, symbol corevus:AOZ1267QI-01
- added C38: 100nF, AlphaLib:0402C, symbol Device:C_Small
- added C97: 2.2nF, AlphaLib:0402C, symbol Device:C_Small
- added C99: 10nF, AlphaLib:0402C, symbol Device:C_Small
- added J43, J44: 1x2P, Connector_PinHeader_2.54mm:PinHeader_1x02_P2.54mm_Vertical, symbol Connector:Conn_01x02_Pin
- added R104: 24kΩ, AlphaLib:0402R, symbol Device:R_Small
- added R109: 22kΩ, AlphaLib:0402R, symbol Device:R_Small
- added R110: 100kΩ, AlphaLib:0402R, symbol Device:R_Small
- added R111, R94, R96: 220kΩ, AlphaLib:0402R, symbol Device:R_Small
- added R112: 4.7kΩ, AlphaLib:0402R, symbol Device:R_Small
- added R91: 5.6kΩ, AlphaLib:0603R, symbol Device:R_Small
- added R95: 18kΩ, AlphaLib:0402R, symbol Device:R_Small
- added U3, U4: TPS54335A, Package_SO:SOIC-8-1EP_3.9x4.9mm_P1.27mm_EP2.95x4.9mm_Mask2.71x3.4mm_ThermalVias, symbol corevus:TPS54335A
- C80: value 1µF -> 100nF
- C88: value 100nF -> 33pF
- C98: value 1µF -> 100pF
- L1: value 6.8μH -> 47μH
- L2: value 4.7μH -> 22μH
- R128: value 4.7kΩ -> 47kΩ
- R129: value 4.7kΩ -> 22kΩ
- R3: value 10kΩ -> 22kΩ
- R3: value 4.7kΩ -> 10kΩ
- R3: value 200kΩ -> 220kΩ
- R90: value 15kΩ -> 30kΩ; footprint AlphaLib:0402R -> AlphaLib:0603R
- R92: value 330kΩ -> 47kΩ; footprint AlphaLib:0402R -> AlphaLib:0603R
- R93: value 330kΩ -> 3.3kΩ; footprint AlphaLib:0402R -> AlphaLib:0603R
- U2: footprint Package_SO:SOP-16_3.9x9.9mm_P1.27mm -> Package_SO:TSSOP-16_4.4x5mm_P0.65mm
Connections:
- net +12V: now also R92.2, J43.1 (Pin_1)
- net +24V: now also R110.1, R94.1, U3.2 (VIN), U4.2 (VIN); no longer R92.1, R93.1
- net +5V: now also J44.1 (Pin_1)
- net GND: now also C88.2, C98.2, R93.1, C97.2, C99.2, J43.2 (Pin_2), J44.2 (Pin_2), R109.2, R111.2, R91.1, R95.2, R96.2, U3.4 (GND), U3.9 (GND), U4.4 (GND), U4.9 (GND); no longer C80.1, C88.1, C98.1
- net H1: now also U1.98 (PC8); no longer U1.96 (PC6)
- net HB: now also U1.96 (PC6); no longer U1.98 (PC8)
- net at L1.1: now also C38.2, U3.3 (PH)
- net at L2.1: now also C80.2, U4.3 (PH)
- net at R90.1: now also R91.2, U4.5 (VSENSE)
- net at R93.2: now also R92.1, U3.5 (VSENSE)
- new net: C80.1, U4.1 (BOOT)
- new net: C98.1, R112.1, U4.6 (COMP)
- new net: R109.1, R110.2, U4.7 (EN)
- new net: R111.1, U4.8 (RT)
- new net: C88.1, R104.1, U3.6 (COMP)
- new net: C97.1, R104.2
- new net: C99.1, R112.2
- new net: R94.2, R95.1, U3.7 (EN)
- new net: C38.1, U3.1 (BOOT)
- new net: R96.1, U3.8 (RT)
- no-connect marks 22 -> 20
Other:
- note added: "0.8V"
- note removed: "EXPERIMENTAl"
- moved on the sheet: C106, C108, C13, C94, C95, D17, D32, L1, L2, R128, R129
