File: hardware/motor_drivers/driver-tmc2209/driver-tmc2209.kicad_sch (KiCad schematic)
At the start: 33 parts, among them M1 JST XH, T10 CS0, T11 STEP, T12 GND, T13 DIR, T14 EN, T17 DIAG, T5 GND, T8 VCC, T9 Therm, U1 TMC2209-LA

Commit message: should be up to date for cvg v0.6 and latest protected drivers
Parts:
- removed M1: JST XH, corevus:XKB_X8821WRS-04, symbol Motor:Stepper_Motor_bipolar
- added C10, C11, C12, C9: 1nF 100V, PCM_ME_passives:0402C, symbol Device:C_Small
- added D3, D4: BAV99S, Package_TO_SOT_SMD:SOT-363_SC-70-6, symbol Diode:BAV99S
- added FB1, FB2, FB3, FB4: 30Ω@100MHz, Resistor_SMD:R_0805_2012Metric, symbol Device:FerriteBead_Small
- added J1: XH, corevus:XH_1x04_SMD_Vertical, symbol Connector_Generic:Conn_01x04
- D1: value G -> Red; footprint AlphaLib:0603LED -> AlphaLib:0402LED
- D2: value Y -> Green; footprint AlphaLib:0603LED -> AlphaLib:0402LED
- H1, H2: footprint corevus:MountingHole_M3_Driver -> corevus:MountingHole_M3_Driver_Corner; now left out of the parts list
- H3: value MountingHole -> Tooling Hole; now left out of the parts list
- H4: value MountingHole -> Tooling Hole; now not fitted; now left out of the parts list
Connections:
- net +24V: now also D3.2 (K2), D3.5 (K4), D4.2 (K2), D4.5 (K4)
- net A1: now also FB2.2
- net A2: now also FB1.2
- net B1: now also FB3.2
- net B2: now also FB4.2
- net GND: now also C10.1, C11.1, C12.1, C9.1, D3.1 (A1), D3.4 (A3), D4.1 (A1), D4.4 (A3)
- new net A1': C10.2, D3.6 (K3A4), FB2.1, J1.2 (Pin_2)
- new net A2': C9.2, D3.3 (K1A2), FB1.1, J1.1 (Pin_1)
- new net B1': C11.2, D4.6 (K3A4), FB3.1, J1.3 (Pin_3)
- new net B2': C12.2, D4.3 (K1A2), FB4.1, J1.4 (Pin_4)
Other:
- moved on the sheet: C13, D1, D2, H1, H2, H3, R1, R16, R20, TH1
