File: hardware/corevus-toolboard/corevus-toolboard.kicad_pcb (KiCad board)
At the start: 4 copper layers, 49.8 x 25.5 mm, 84 parts, among them J1 MF3, J10 1x3P, J2 XH, J3 MF3, J4 XH, J5 XH, J6 XH, J7 XH, J8 pinheader, J9 XH, Q2 NMOS, Q4 AO3400, SW1 RST, U1 LIS2DE12, U2 TPS54302, U3 STM32G431KBU3, U4 TMC2209-LA, U6 SPX3819M5-L-3-3, U7 TPS2069CDBV, U8 UCC27517, Y1 XRCGB25

Commit message: cleaned up corevus toolboard schematics to be more presentable
Parts:
- C2, C3: value 10pF -> 6pF
- C23: value 100nF 50V -> 100nF 50V
- C28: value 68pF -> 68pF
- C7: value 100nF -> 100nF
- J1: value MF3 -> MF3 1x2P
- J2, J5, J6, J7, J9: value XH -> XH 1x2P
- J3: value MF3 -> MX3.0 2x4P
- J4: value XH -> XH 1x4P
- J8: value pinheader -> 1x8P
- SW1: value RST -> Reset
- turned C23 to 180 degrees
- turned R21 to 180 degrees
Connections:
- C23 pad 1: Net-(J6-Pin_1) -> /PCF_V+
- C23 pad 2: /PCF_V+ -> Net-(J6-Pin_1)
- R21 pad 1: /~{En} -> Net-(D3-K)
- R21 pad 2: Net-(D3-K) -> /~{En}
- U4 pad 11: /Diag -> unconnected-(U4-DIAG-Pad11)
Changed lines of the file:
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@@
 	(net 34 "unconnected-(U4-MS1-Pad9)")
 	(net 35 "unconnected-(U4-MS2-Pad10)")
-	(net 36 "/Diag")
+	(net 36 "unconnected-(U4-DIAG-Pad11)")
 	(net 37 "unconnected-(U4-INDEX-Pad12)")
 	(net 38 "unconnected-(U4-CLK-Pad13)")
@@
 			)
 		)
-		(property "Value" "pinheader"
+		(property "Value" "1x8P"
 			(at -1.17 19 0)
 			(layer "F.Fab")
@@
 			)
 		)
-		(property "Value" "MF3"
+		(property "Value" "MF3 1x2P"
 			(at 0 -1.5 90)
 			(layer "F.Fab")
@@
 			)
 		)
-		(property "Value" "XH"
+		(property "Value" "XH 1x2P"
 			(at 0 2.75 90)
 			(layer "F.Fab")
@@
 			)
 		)
-		(property "Description" ""
+		(property "Description" "Generic connector, single row, 01x03, script generated (kicad-library-utils/schlib/autogen/connector/)"
 			(at 0 0 90)
 			(layer "F.Fab")
@@
 			)
 		)
-		(property "Value" "XH"
+		(property "Value" "XH 1x4P"
 			(at 0 -4 -90)
 			(unlocked yes)
@@
 			)
 		)
-		(property "Description" ""
+		(property "Description" "Generic connector, single row, 01x04, script generated (kicad-library-utils/schlib/autogen/connector/)"
 			(at 0 0 -90)
 			(unlocked yes)
@@
 			)
 		)
-		(property "Value" "XH"
+		(property "Value" "XH 1x2P"
 			(at 0 2.75 90)
 			(layer "F.Fab")
@@
 			)
 		)
-		(property "Description" ""
+		(property "Description" "Generic connector, single row, 01x02, script generated (kicad-library-utils/schlib/autogen/connector/)"
 			(at 0 0 90)
 			(layer "F.Fab")
@@
 			)
 		)
-		(property "Value" "XH"
+		(property "Value" "XH 1x2P"
 			(at 0 2.75 90)
 			(layer "F.Fab")
@@
 			)
 		)
-		(property "Description" ""
+		(property "Description" "Generic connector, single row, 01x03, script generated (kicad-library-utils/schlib/autogen/connector/)"
 			(at 0 0 90)
 			(layer "F.Fab")
@@
 			)
 		)
-		(property "Value" "XH"
+		(property "Value" "XH 1x2P"
 			(at 0 2.75 90)
 			(layer "F.Fab")
@@
 			)
 		)
-		(property "Description" ""
+		(property "Description" "Generic connector, single row, 01x02, script generated (kicad-library-utils/schlib/autogen/connector/)"
 			(at 0 0 90)
 			(layer "F.Fab")
@@
 			)
 		)
-		(property "Value" "XH"
+		(property "Value" "XH 1x2P"
 			(at 0 2.75 90)
 			(layer "F.Fab")
@@
 			)
 		)
-		(property "Description" ""
+		(property "Description" "Generic connector, single row, 01x02, script generated (kicad-library-utils/schlib/autogen/connector/)"
 			(at 0 0 90)
 			(layer "F.Fab")
@@
 			)
 		)
-		(property "Value" "MF3"
+		(property "Value" "MX3.0 2x4P"
 			(at 0 -4.950001 0)
 			(layer "F.Fab")
@@
 		(fp_arc
 			(start -1.515545 0.875)
-			(mid -1.750004 -0.000001)
+			(mid -1.750004 0)
 			(end -1.515544 -0.875)
 			(stroke
@@
 			)
 		)
-		(property "Value" "RST"
+		(property "Value" "Reset"
 			(at 0 -0.75 0)
 			(layer "B.Fab")
@@
 		(sheetfile "corevus-toolboard.kicad_sch")
 		(zone_connect 1)
-		(attr exclude_from_pos_files exclude_from_bom)
+		(attr exclude_from_pos_files)
 		(fp_line
 			(start 1.4 -0.300001)
@@
 	(footprint "AlphaLib:0402R"
 		(layer "B.Cu")
-		(at 9.5 -6)
+		(at 9.5 -6 180)
 		(descr "Capacitor 0402 package")
 		(tags "capacitor cap")
@@
 		(attr smd)
 		(fp_line
-			(start -0.1 -0.15)
-			(end 0.1 -0.15)
+			(start -0.1 0.15)
+			(end 0.1 0.15)
 			(stroke
 				(width 0.1)
@@
 		)
 		(fp_line
-			(start -0.1 0.15)
-			(end 0.1 0.15)
+			(start -0.1 -0.15)
+			(end 0.1 -0.15)
 			(stroke
 				(width 0.1)
@@
 		)
 		(fp_line
-			(start -0.9 -0.499999)
-			(end 0.9 -0.499999)
+			(start 0.9 0.499999)
+			(end -0.9 0.499999)
 			(stroke
 				(width 0.05)
@@
 		)
 		(fp_line
-			(start -0.9 0.499999)
-			(end -0.9 -0.499999)
+			(start 0.9 -0.499999)
+			(end 0.9 0.499999)
 			(stroke
 				(width 0.05)
@@
 		)
 		(fp_line
-			(start 0.9 -0.499999)
-			(end 0.9 0.499999)
+			(start -0.9 0.499999)
+			(end -0.9 -0.499999)
 			(stroke
 				(width 0.05)
@@
 		)
 		(fp_line
-			(start 0.9 0.499999)
-			(end -0.9 0.499999)
+			(start -0.9 -0.499999)
+			(end 0.9 -0.499999)
 			(stroke
 				(width 0.05)
@@
 		)
 		(pad "1" smd roundrect
-			(at -0.499999 0)
+			(at -0.499999 0 180)
 			(size 0.55 0.6)
 			(layers "B.Cu" "B.Paste" "B.Mask")
 			(roundrect_rratio 0.1818181818)
-			(net 32 "/~{En}")
+			(net 59 "Net-(D3-K)")
 			(pintype "passive")
 		)
 		(pad "2" smd roundrect
-			(at 0.499999 0)
+			(at 0.499999 0 180)
 			(size 0.55 0.6)
 			(layers "B.Cu" "B.Paste" "B.Mask")
 			(roundrect_rratio 0.1818181818)
-			(net 59 "Net-(D3-K)")
+			(net 32 "/~{En}")
 			(pintype "passive")
 		)
@@
 		(tags "capacitor cap")
 		(property "Reference" "R8"
-			(at 0 0.9 360)
+			(at 0 0.9 0)
 			(layer "B.SilkS")
 			(hide yes)
@@
 		)
 		(property "Value" "2.2kΩ"
-			(at 0 -0.1 360)
+			(at 0 -0.1 0)
 			(layer "B.Fab")
 			(effects
@@
 		)
 		(property "Footprint" "AlphaLib:0402R"
-			(at 0 0 360)
+			(at 0 0 0)
 			(layer "B.Fab")
 			(hide yes)
@@
 		)
 		(property "Datasheet" ""
-			(at 0 0 360)
+			(at 0 0 0)
 			(layer "B.Fab")
 			(hide yes)
@@
 		)
 		(property "Description" ""
-			(at 0 0 360)
+			(at 0 0 0)
 			(layer "B.Fab")
 			(hide yes)
@@
 		)
 		(fp_text user "${REFERENCE}"
-			(at 0 0.15 360)
+			(at 0 0.15 0)
 			(layer "B.Fab")
 			(effects
@@
 			)
 		)
-		(property "Value" "10pF"
+		(property "Value" "6pF"
 			(at 0 -0.1 0)
 			(layer "B.Fab")
@@
 			(layers "B.Cu" "B.Paste" "B.Mask")
 			(roundrect_rratio 0.25)
-			(net 36 "/Diag")
+			(net 36 "unconnected-(U4-DIAG-Pad11)")
 			(pinfunction "DIAG")
-			(pintype "output")
+			(pintype "output+no_connect")
 		)
 		(pad "12" smd roundrect
@@
 			)
 		)
-		(property "Value" "68pF "
+		(property "Value" "68pF"
 			(at 0 -0.1 0)
 			(layer "B.Fab")
@@
 			)
 		)
-		(property "Value" "10pF"
+		(property "Value" "6pF"
 			(at 0 -0.1 0)
 			(layer "B.Fab")
@@
 	(footprint "AlphaLib:0402C"
 		(layer "B.Cu")
-		(at -9.5 -3.75)
+		(at -9.5 -3.75 180)
 		(descr "Capacitor 0402 package")
 		(tags "capacitor cap")
 		(property "Reference" "C23"
-			(at 0 0.9 0)
+			(at 0 0.9 360)
 			(layer "B.SilkS")
 			(hide yes)
@@
 			)
 		)
-		(property "Value" " 100nF 50V"
-			(at 0 -0.1 0)
+		(property "Value" "100nF 50V"
+			(at 0 -0.1 360)
 			(layer "B.Fab")
 			(effects
@@
 		)
 		(property "Footprint" "AlphaLib:0402C"
-			(at 0 0 0)
+			(at 0 0 360)
 			(layer "B.Fab")
 			(hide yes)
@@
 		)
 		(property "Datasheet" ""
-			(at 0 0 0)
+			(at 0 0 360)
 			(layer "B.Fab")
 			(hide yes)
@@
 		)
 		(property "Description" ""
-			(at 0 0 0)
+			(at 0 0 360)
 			(layer "B.Fab")
 			(hide yes)
@@
 		(attr smd)
 		(fp_line
-			(start -0.1 0.2)
-			(end -0.1 -0.2)
+			(start 0.1 0.2)
+			(end 0.1 -0.2)
 			(stroke
 				(width 0.1)
@@
 		)
 		(fp_line
-			(start 0.1 0.2)
-			(end 0.1 -0.2)
+			(start -0.1 0.2)
+			(end -0.1 -0.2)
 			(stroke
 				(width 0.1)
@@
 		)
 		(fp_line
-			(start -0.9 -0.499999)
-			(end 0.9 -0.499999)
+			(start 0.9 0.499999)
+			(end -0.9 0.499999)
 			(stroke
 				(width 0.05)
@@
 		)
 		(fp_line
-			(start -0.9 0.499999)
-			(end -0.9 -0.499999)
+			(start 0.9 -0.499999)
+			(end 0.9 0.499999)
 			(stroke
 				(width 0.05)
@@
 		)
 		(fp_line
-			(start 0.9 -0.499999)
-			(end 0.9 0.499999)
+			(start -0.9 0.499999)
+			(end -0.9 -0.499999)
 			(stroke
 				(width 0.05)
@@
 		)
 		(fp_line
-			(start 0.9 0.499999)
-			(end -0.9 0.499999)
+			(start -0.9 -0.499999)
+			(end 0.9 -0.499999)
 			(stroke
 				(width 0.05)
@@
 		)
 		(fp_text user "${REFERENCE}"
-			(at 0 0.15 0)
+			(at 0 0.15 360)
 			(layer "B.Fab")
 			(effects
@@
 		)
 		(pad "1" smd roundrect
-			(at -0.499999 0)
+			(at -0.499999 0 180)
 			(size 0.55 0.6)
 			(layers "B.Cu" "B.Paste" "B.Mask")
 			(roundrect_rratio 0.1818181818)
-			(net 26 "Net-(J6-Pin_1)")
+			(net 48 "/PCF_V+")
 			(pintype "passive")
 		)
 		(pad "2" smd roundrect
-			(at 0.499999 0)
+			(at 0.499999 0 180)
 			(size 0.55 0.6)
 			(layers "B.Cu" "B.Paste" "B.Mask")
 			(roundrect_rratio 0.1818181818)
-			(net 48 "/PCF_V+")
+			(net 26 "Net-(J6-Pin_1)")
 			(pintype "passive")
 		)
@@
 		(tags "capacitor cap")
 		(property "Reference" "R1"
-			(at 0 0.9 360)
+			(at 0 0.9 0)
 			(layer "B.SilkS")
 			(hide yes)
@@
 		)
 		(property "Value" "4.7kΩ"
-			(at 0 -0.1 360)
+			(at 0 -0.1 0)
 			(layer "B.Fab")
 			(effects
@@
 		)
 		(property "Footprint" "AlphaLib:0402R"
-			(at 0 0 360)
+			(at 0 0 0)
 			(layer "B.Fab")
 			(hide yes)
@@
 		)
 		(property "Datasheet" ""
-			(at 0 0 360)
+			(at 0 0 0)
 			(layer "B.Fab")
 			(hide yes)
@@
 		)
 		(property "Description" ""
-			(at 0 0 360)
+			(at 0 0 0)
 			(layer "B.Fab")
 			(hide yes)
@@
 		)
 		(fp_text user "${REFERENCE}"
-			(at 0 0.15 360)
+			(at 0 0.15 0)
 			(layer "B.Fab")
 			(effects
@@
 			)
 		)
-		(property "Value" "100nF "
+		(property "Value" "100nF"
 			(at 0 -0.1 90)
 			(layer "B.Fab")
@@
 		(fp_arc
 			(start -1.515545 0.875)
-			(mid -1.750004 -0.000001)
+			(mid -1.750004 0)
 			(end -1.515544 -0.875)
 			(stroke

Commit message: update toolboard, change documentation
Parts:
- C2, C3: value 6pF -> 10pF
- J2, J9: value XH 1x2P -> XH 1x3P
Routing:
- net +3.3V: track 86.4 -> 83.7 mm, vias 8 -> 6
- net /BOOT0: track 23.7 -> 23.1 mm, vias 3 -> 2
- net /PA5: track 23.5 -> 24.0 mm, vias 0 -> 1
- net /PA6: track 25.2 -> 25.7 mm, vias 0 -> 1
- net /PA4: track 31.9 -> 31.6 mm, vias 0 -> 2
- net /PA7: track 26.9 -> 27.0 mm, vias 0 -> 1
- net GND: vias 83 -> 82
Other:
- board text added: "MERIDI ENGINEERING SEP 2024 COREVUS TOOLBOARD v1.0"
- board text added: "PA4"
- board text added: "PA5"
- board text added: "PA6"
- board text added: "PA7"
- board text added: "PB8"
- board text added: "TOOLBOARD v1.0"
- board text removed: "A4"
- board text removed: "A5"
- board text removed: "A6"
- board text removed: "A7"
- board text removed: "B8"
- board text removed: "MERIDI ENGINEERING JULY 2024 COREVUS TOOLBOARD v0.3"
- board text removed: "TOOLBOARD v0.3"
