File: hardware/corevus-toolboard/corevus-toolboard.kicad_sch (KiCad schematic)
At the start: 87 parts, among them J1 MF3 1x2P, J10 1x3P, J2 XH 1x2P, J3 MX3.0 2x4P, J4 XH 1x4P, J5 XH 1x2P, J6 XH 1x2P, J7 XH 1x2P, J8 1x8P, J9 XH 1x2P, Q2 NMOS, Q4 AO3400, SW3 Reset, U1 LIS2DE12, U2 TPS54302, U3 STM32G431KBU3, U4 TMC2209-LA, U6 SPX3819M5-L-3-3, U7 TPS2069CDBV, U8 UCC27517, Y1 XRCGB25

Commit message: update toolboard, change documentation
Parts:
- J2, J9: value XH 1x2P -> XH 1x3P
Other:
- moved on the sheet: C2, C3, SW3
Changed lines of the file:
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@@
 	)
 	(junction
-		(at 26.67 40.64)
-		(diameter 0)
-		(color 0 0 0 0)
-	)
-	(junction
 		(at 167.64 26.67)
 		(diameter 0)
@@
 	)
 	(junction
-		(at 26.67 44.45)
+		(at 57.15 81.28)
 		(diameter 0)
 		(color 0 0 0 0)
 	)
 	(junction
-		(at 57.15 81.28)
+		(at 191.77 106.68)
 		(diameter 0)
 		(color 0 0 0 0)
 	)
 	(junction
-		(at 191.77 106.68)
+		(at 180.34 76.2)
 		(diameter 0)
 		(color 0 0 0 0)
 	)
 	(junction
-		(at 180.34 76.2)
+		(at 27.94 44.45)
 		(diameter 0)
 		(color 0 0 0 0)
@@
 	)
 	(junction
+		(at 27.94 40.64)
+		(diameter 0)
+		(color 0 0 0 0)
+	)
+	(junction
 		(at 46.99 22.86)
 		(diameter 0)
@@
 	(wire
 		(pts
-			(xy 26.67 36.83) (xy 26.67 40.64)
+			(xy 27.94 36.83) (xy 27.94 40.64)
 		)
 		(stroke
@@
 	(wire
 		(pts
-			(xy 34.29 33.02) (xy 40.64 33.02)
-		)
-		(stroke
-			(width 0)
-			(type default)
-		)
-	)
-	(wire
-		(pts
 			(xy 256.54 26.67) (xy 256.54 27.94)
 		)
@@
 	(wire
 		(pts
-			(xy 26.67 40.64) (xy 30.48 40.64)
-		)
-		(stroke
-			(width 0)
-			(type default)
-		)
-	)
-	(wire
-		(pts
 			(xy 222.25 106.68) (xy 224.79 106.68)
 		)
@@
 	(wire
 		(pts
-			(xy 31.75 36.83) (xy 33.02 36.83)
+			(xy 27.94 40.64) (xy 30.48 40.64)
 		)
 		(stroke
@@
 	(wire
 		(pts
-			(xy 26.67 44.45) (xy 26.67 40.64)
+			(xy 27.94 44.45) (xy 27.94 40.64)
 		)
 		(stroke
@@
 		)
 	)
-	(wire
-		(pts
-			(xy 31.75 44.45) (xy 33.02 44.45)
-		)
-		(stroke
-			(width 0)
-			(type default)
-		)
-	)
 	(polyline
 		(pts
@@
 	(wire
 		(pts
-			(xy 25.4 44.45) (xy 26.67 44.45)
+			(xy 25.4 44.45) (xy 27.94 44.45)
 		)
 		(stroke
@@
 	(wire
 		(pts
+			(xy 35.56 33.02) (xy 40.64 33.02)
+		)
+		(stroke
+			(width 0)
+			(type default)
+		)
+	)
+	(wire
+		(pts
 			(xy 44.45 22.86) (xy 46.99 22.86)
 		)
@@
 	)
 	(label "~{Reset}"
-		(at 34.29 33.02 0)
+		(at 39.37 33.02 180)
 		(fields_autoplaced yes)
 		(effects
@@
 				(size 1.27 1.27)
 			)
-			(justify left bottom)
+			(justify right bottom)
 		)
 	)
@@
 			)
 		)
-		(property "Value" "XH 1x2P"
+		(property "Value" "XH 1x3P"
 			(at 158.75 101.6 0)
 			(effects
@@
 	(symbol
 		(lib_id "Device:C_Small")
-		(at 29.21 36.83 270)
+		(at 30.48 36.83 270)
 		(unit 1)
 		(exclude_from_sim no)
@@
 		(dnp no)
 		(property "Reference" "C2"
-			(at 30.21 35.83 90)
+			(at 31.48 35.83 90)
 			(effects
 				(font
@@
 		)
 		(property "Value" "10pF"
-			(at 28.21 35.83 90)
+			(at 29.48 35.83 90)
 			(effects
 				(font
@@
 		)
 		(property "Footprint" "AlphaLib:0402C"
-			(at 29.21 36.83 0)
+			(at 30.48 36.83 0)
 			(effects
 				(font
@@
 		)
 		(property "Datasheet" "~"
-			(at 29.21 36.83 0)
+			(at 30.48 36.83 0)
 			(effects
 				(font
@@
 		)
 		(property "Description" ""
-			(at 29.21 36.83 0)
+			(at 30.48 36.83 0)
 			(effects
 				(font
@@
 		(dnp no)
 		(property "Reference" "Y1"
-			(at 26.416 39.37 90)
+			(at 26.67 39.37 90)
 			(effects
 				(font
@@
 		)
 		(property "Value" "XRCGB25"
-			(at 26.416 41.91 90)
+			(at 26.67 41.91 90)
 			(effects
 				(font
@@
 			)
 		)
-		(property "Value" "XH 1x2P"
+		(property "Value" "XH 1x3P"
 			(at 179.07 101.6 0)
 			(effects
@@
 	(symbol
 		(lib_id "Switch:SW_Push")
-		(at 29.21 33.02 0)
+		(at 30.48 33.02 0)
 		(mirror y)
 		(unit 1)
@@
 		(dnp no)
 		(property "Reference" "SW3"
-			(at 29.21 26.162 0)
+			(at 30.48 26.162 0)
 			(effects
 				(font
@@
 		)
 		(property "Value" "Reset"
-			(at 29.21 28.702 0)
+			(at 30.48 28.702 0)
 			(effects
 				(font
@@
 		)
 		(property "Footprint" "corevus:ShouHan_TS24CA"
-			(at 29.21 27.94 0)
+			(at 30.48 27.94 0)
 			(effects
 				(font
@@
 		)
 		(property "Datasheet" "~"
-			(at 29.21 27.94 0)
+			(at 30.48 27.94 0)
 			(effects
 				(font
@@
 		)
 		(property "Description" ""
-			(at 29.21 33.02 0)
+			(at 30.48 33.02 0)
 			(effects
 				(font
@@
 	(symbol
 		(lib_id "power:GND")
-		(at 24.13 33.02 270)
+		(at 25.4 33.02 270)
 		(unit 1)
 		(exclude_from_sim no)
@@
 		(dnp no)
 		(property "Reference" "#PWR0150"
-			(at 17.78 33.02 0)
+			(at 19.05 33.02 0)
 			(effects
 				(font
@@
 		)
 		(property "Value" "GND"
-			(at 21.59 33.02 90)
+			(at 22.86 33.02 90)
 			(effects
 				(font
@@
 		)
 		(property "Footprint" ""
-			(at 24.13 33.02 0)
+			(at 25.4 33.02 0)
 			(effects
 				(font
@@
 		)
 		(property "Datasheet" ""
-			(at 24.13 33.02 0)
+			(at 25.4 33.02 0)
 			(effects
 				(font
@@
 		)
 		(property "Description" ""
-			(at 24.13 33.02 0)
+			(at 25.4 33.02 0)
 			(effects
 				(font
@@
 	(symbol
 		(lib_id "Device:C_Small")
-		(at 29.21 44.45 270)
+		(at 30.48 44.45 270)
 		(mirror x)
 		(unit 1)
@@
 		(dnp no)
 		(property "Reference" "C3"
-			(at 30.21 45.45 90)
+			(at 31.48 45.45 90)
 			(effects
 				(font
@@
 		)
 		(property "Value" "10pF"
-			(at 28.21 45.45 90)
+			(at 29.48 45.45 90)
 			(effects
 				(font
@@
 		)
 		(property "Footprint" "AlphaLib:0402C"
-			(at 29.21 44.45 0)
+			(at 30.48 44.45 0)
 			(effects
 				(font
@@
 		)
 		(property "Datasheet" "~"
-			(at 29.21 44.45 0)
+			(at 30.48 44.45 0)
 			(effects
 				(font
@@
 		)
 		(property "Description" ""
-			(at 29.21 44.45 0)
+			(at 30.48 44.45 0)
 			(effects
 				(font
